Commit message: create DAE and STL folder

File: urdf/sensor/hokuyo_utm30lx.urdf.xacro (robot description, xacro)
@@ -18,5 +18,5 @@
           <origin xyz="0 0 0" rpy="0 0 0" />
           <geometry>
-          <mesh filename="package://ubiquitous_display_description/meshes/hokuyo_utm_30lx.dae"/>
+          <mesh filename="package://ubiquitous_display_description/meshes/DAE/hokuyo_utm_30lx.dae"/>
         </geometry>
         </visual>

File: urdf/sensor/kinect2.urdf.xacro (robot description, xacro)
@@ -13,5 +13,5 @@
         <geometry>
           <!-- these meshes were exported in mm, so scale back to m -->
-          <mesh filename="package://ubiquitous_display_description/meshes/kinect2_origin_on_rgb_optical_frame.stl" scale="0.001 0.001 0.001"/>
+          <mesh filename="package://ubiquitous_display_description/meshes/STL/kinect2_origin_on_rgb_optical_frame.stl" scale="0.001 0.001 0.001"/>
         </geometry>
         <material name="Kinect2Grey"/>

File: urdf/ubiquitous_display.urdf.xacro (robot description, xacro)
@@ -36,5 +36,5 @@
       <geometry>
           <!-- these meshes were exported in mm, so scale back to m -->
-        <mesh filename="package://ubiquitous_display_description/meshes/kinect2_origin_on_rgb_optical_frame.stl" scale="0.001 0.001 0.001"/>
+        <mesh filename="package://ubiquitous_display_description/meshes/STL/kinect2_origin_on_rgb_optical_frame.stl" scale="0.001 0.001 0.001"/>
         <!--box size="0.25 0.07 0.45" /-->
       </geometry>

File: urdf/youbot/base.urdf.xacro (robot description, xacro)
@@ -48,5 +48,5 @@
         <origin xyz="0 0 0" rpy="0 0 0"/>
         <geometry>
-          <mesh filename="package://ubiquitous_display_description/meshes/base.dae"/>
+          <mesh filename="package://ubiquitous_display_description/meshes/DAE/base.dae"/>
         </geometry>
         <material name="DarkGrey"/>
@@ -56,5 +56,5 @@
         <geometry>
           <!--<box size="${base_size_x} ${base_size_y} ${base_size_z}" />-->
-          <mesh filename="package://ubiquitous_display_description/meshes/base_convex.dae"/>
+          <mesh filename="package://ubiquitous_display_description/meshes/DAE/base_convex.dae"/>
         </geometry>
       </collision>
