Commit message: fixed pantilt.gazebo and pantilt.transmission

File: urdf/pantilt/pantilt.transmission.xacro (robot description, xacro)
@@ -2,24 +2,25 @@
 <robot name="pantilt_trans" xmlns:xacro="http://ros.org/wiki/xacro">
 <xacro:macro name="ubiquitous_display_transmission">
-<transmission name="pan_tran">
-  <type>transmission_interface/SimpleTransmission</type>
-  <joint name="pan_joint">
-    <hardwareInterface>hardware_interface/EffortJointInterface</hardwareInterface>
-  </joint>
-  <actuator name="pan_motor">
-    <hardwareInterface>hardware_interface/EffortJointInterface</hardwareInterface>
-    <mechanicalReduction>1</mechanicalReduction>
-  </actuator>
-</transmission>
-<transmission name="tilt_tran">
-  <type>transmission_interface/SimpleTransmission</type>
-  <joint name="tilt_joint">
-    <hardwareInterface>hardware_interface/EffortJointInterface</hardwareInterface>
-  </joint>
-  <actuator name="tilt_motor">
-    <hardwareInterface>hardware_interface/EffortJointInterface</hardwareInterface>
-    <mechanicalReduction>1</mechanicalReduction>
-  </actuator>
-</transmission>
+  <transmission name="trans1">
+    <type>transmission_interface/SimpleTransmission</type>
+    <joint name="pan_joint">
+      <hardwareInterface>hardware_interface/EffortJointInterface</hardwareInterface>
+    </joint>
+    <actuator name="motor1">
+      <hardwareInterface>hardware_interface/EffortJointInterface</hardwareInterface>
+      <mechanicalReduction>1</mechanicalReduction>
+    </actuator>
+  </transmission>
+  <transmission name="tran2">
+    <type>transmission_interface/SimpleTransmission</type>
+    <joint name="tilt_joint">
+      <hardwareInterface>hardware_interface/EffortJointInterface</hardwareInterface>
+    </joint>
+    <actuator name="motor2">
+      <hardwareInterface>hardware_interface/EffortJointInterface</hardwareInterface>
+      <mechanicalReduction>1</mechanicalReduction>
+    </actuator>
+  </transmission>
 </xacro:macro>
+<xacro:ubiquitous_display_transmission />
 </robot>

File: urdf/youbot/base.transmission.xacro (robot description, xacro)
@@ -12,9 +12,9 @@
 			<type>transmission_interface/SimpleTransmission</type>
 			<actuator name="wheel_motor_fl">
-				<hardwareInterface>VelocityJointInterface</hardwareInterface>
+				<hardwareInterface>hardware_interface/VelocityJointInterface</hardwareInterface>
 				<mechanicalReduction>${wheel_mechanical_reduction}</mechanicalReduction>
 			</actuator>
 			<joint name="wheel_joint_fl">
-				<hardwareInterface>VelocityJointInterface</hardwareInterface>
+				<hardwareInterface>hardware_interface/VelocityJointInterface</hardwareInterface>
 			</joint>
 		</transmission>
@@ -22,9 +22,9 @@
 			<type>transmission_interface/SimpleTransmission</type>
 			<actuator name="caster_motor_fl">
-				<hardwareInterface>VelocityJointInterface</hardwareInterface>
+				<hardwareInterface>hardware_interface/VelocityJointInterface</hardwareInterface>
 				<mechanicalReduction>${caster_mechanical_reduction}</mechanicalReduction>
 			</actuator>
 			<joint name="caster_joint_fl">
-				<hardwareInterface>VelocityJointInterface</hardwareInterface>
+				<hardwareInterface>hardware_interface/VelocityJointInterface</hardwareInterface>
 			</joint>
 		</transmission>
@@ -33,9 +33,9 @@
 			<type>transmission_interface/SimpleTransmission</type>
 			<actuator name="wheel_motor_fr">
-				<hardwareInterface>VelocityJointInterface</hardwareInterface>
+				<hardwareInterface>hardware_interface/VelocityJointInterface</hardwareInterface>
 				<mechanicalReduction>${wheel_mechanical_reduction}</mechanicalReduction>
 			</actuator>
 			<joint name="wheel_joint_fr">
-				<hardwareInterface>VelocityJointInterface</hardwareInterface>
+				<hardwareInterface>hardware_interface/VelocityJointInterface</hardwareInterface>
 			</joint>
 		</transmission>
@@ -43,9 +43,9 @@
 			<type>transmission_interface/SimpleTransmission</type>
 			<actuator name="caster_motor_fr" >
-				<hardwareInterface>VelocityJointInterface</hardwareInterface>
+				<hardwareInterface>hardware_interface/VelocityJointInterface</hardwareInterface>
 				<mechanicalReduction>${caster_mechanical_reduction}</mechanicalReduction>
 			</actuator>
 			<joint name="caster_joint_fr">
-				<hardwareInterface>VelocityJointInterface</hardwareInterface>
+				<hardwareInterface>hardware_interface/VelocityJointInterface</hardwareInterface>
 			</joint>
 		</transmission>
@@ -54,9 +54,9 @@
 			<type>transmission_interface/SimpleTransmission</type>
 			<actuator name="wheel_motor_bl" >
-				<hardwareInterface>VelocityJointInterface</hardwareInterface>
+				<hardwareInterface>hardware_interface/VelocityJointInterface</hardwareInterface>
 				<mechanicalReduction>${wheel_mechanical_reduction}</mechanicalReduction>
 			</actuator>
 			<joint name="wheel_joint_bl">
-				<hardwareInterface>VelocityJointInterface</hardwareInterface>
+				<hardwareInterface>hardware_interface/VelocityJointInterface</hardwareInterface>
 			</joint>
 		</transmission>
@@ -64,9 +64,9 @@
 			<type>transmission_interface/SimpleTransmission</type>
 			<actuator name="caster_motor_bl" >
-				<hardwareInterface>VelocityJointInterface</hardwareInterface>
+				<hardwareInterface>hardware_interface/VelocityJointInterface</hardwareInterface>
 				<mechanicalReduction>${caster_mechanical_reduction}</mechanicalReduction>
 			</actuator>
 			<joint name="caster_joint_bl">
-				<hardwareInterface>VelocityJointInterface</hardwareInterface>
+				<hardwareInterface>hardware_interface/VelocityJointInterface</hardwareInterface>
 			</joint>
 		</transmission>
@@ -75,9 +75,9 @@
 			<type>transmission_interface/SimpleTransmission</type>
 			<actuator name="wheel_motor_br" >
-				<hardwareInterface>VelocityJointInterface</hardwareInterface>
+				<hardwareInterface>hardware_interface/VelocityJointInterface</hardwareInterface>
 				<mechanicalReduction>${wheel_mechanical_reduction}</mechanicalReduction>
 			</actuator>
 			<joint name="wheel_joint_br">
-				<hardwareInterface>VelocityJointInterface</hardwareInterface>
+				<hardwareInterface>hardware_interface/VelocityJointInterface</hardwareInterface>
 			</joint>
 		</transmission>
@@ -85,9 +85,9 @@
 			<type>transmission_interface/SimpleTransmission</type>
 			<actuator name="caster_motor_br" >
-				<hardwareInterface>VelocityJointInterface</hardwareInterface>
+				<hardwareInterface>hardware_interface/VelocityJointInterface</hardwareInterface>
 				<mechanicalReduction>${caster_mechanical_reduction}</mechanicalReduction>
 			</actuator>
 			<joint name="caster_joint_br">
-				<hardwareInterface>VelocityJointInterface</hardwareInterface>
+				<hardwareInterface>hardware_interface/VelocityJointInterface</hardwareInterface>
 			</joint>
 		</transmission>
