Commit message: add gazebo tag

File: urdf/pantilt/pantilt.gazebo.xacro (robot description, xacro)
@@ -15,4 +15,14 @@
     <material>Gazebo/Grey</material>
   </gazebo>
+  <gazebo reference="left_pt_pillars">
+    <mu1>0.2</mu1>
+    <mu2>0.2</mu2>
+    <material>Gazebo/Grey</material>
+  </gazebo>
+  <gazebo reference="right_pt_pillars">
+    <mu1>0.2</mu1>
+    <mu2>0.2</mu2>
+    <material>Gazebo/Grey</material>
+  </gazebo>
 </xacro:macro>
   <xacro:pantilt_gazebo name="ud_pt_"/>

File: urdf/pantilt/pantilt.urdf.xacro (robot description, xacro)
@@ -62,4 +62,12 @@
         <material name="gray" />
       </visual>
+     <inertial>
+       <origin xyz="0 0 0.01" rpy="0 0 0"/>
+       <mass value="1"/>
+       <inertia
+	    ixx="1.0" ixy="0.0" ixz="0.0"
+	    iyy="1.0" iyz="0.0"
+	    izz="1.0"/>
+     </inertial>
     </link>
     <link name="right_pt_pillars" >
@@ -71,4 +79,12 @@
         <material name="gray" />
       </visual>
+     <inertial>
+       <origin xyz="0 0 0.01" rpy="0 0 0"/>
+       <mass value="1"/>
+       <inertia
+	    ixx="1.0" ixy="0.0" ixz="0.0"
+	    iyy="1.0" iyz="0.0"
+	    izz="1.0"/>
+     </inertial>
     </link>
     <link name="${name}projector_link">
