Commit message: add pantilt.gazebo.xacro

File: urdf/pantilt/pantilt.urdf.xacro (robot description, xacro)
@@ -19,6 +19,5 @@
     </link>
     <link name="${name}box_link" >
-      <visual>down processing monitor complete
-done
+      <visual>
         <origin xyz="0 0 0" rpy="0 0 0" />
         <geometry>

Commit message: add <collision> in pantilt.urdf.xacro

File: urdf/pantilt/pantilt.urdf.xacro (robot description, xacro)
@@ -21,4 +21,10 @@
     </link>
     <link name="${name}box_link" >
+      <collision>
+        <origin xyz="0 0 0.0325" rpy="0 0 0"/>
+        <geometry>
+          <box size="0.07 0.085 0.065"/>
+        </geometry>
+      </collision>
       <visual>
         <origin xyz="0 0 0" rpy="0 0 0" />
@@ -38,4 +44,10 @@
     </link>
     <link name="${name}plate_link">
+      <collision>
+        <origin xyz="0 0 0.0015" rpy="0 0 0"/>
+        <geometry>
+          <box size="0.35 0.095 0.003"/>
+        </geometry>
+      </collision>
       <visual>
         <origin xyz="-0.075 0 0" rpy="0 0 0" />
@@ -55,4 +67,10 @@
     </link>
     <link name="left_pt_pillars" >
+      <collision>
+        <origin xyz="0 0 0.10" rpy="0 0 0"/>
+        <geometry>
+          <box size="0.01 0.05 0.20"/>
+        </geometry>
+      </collision>
       <visual>
         <origin xyz="0 0 0" rpy="0 0 0" />
@@ -72,4 +90,10 @@
     </link>
     <link name="right_pt_pillars" >
+      <collision>
+        <origin xyz="0 0 0.10" rpy="0 0 0"/>
+        <geometry>
+          <box size="0.01 0.05 0.20"/>
+        </geometry>
+      </collision>
       <visual>
         <origin xyz="0 0 0" rpy="0 0 0" />
@@ -89,4 +113,10 @@
     </link>
     <link name="${name}projector_link">
+      <collision>
+        <origin xyz="0 0 0.035" rpy="0 0 0"/>
+        <geometry>
+          <box size="0.24 0.17 0.07"/>
+        </geometry>
+      </collision>
       <visual>
         <origin xyz="0.07 0.037 0" rpy="0 0 0" />

Commit message: calcurate inertial

File: urdf/pantilt/pantilt.urdf.xacro (robot description, xacro)
@@ -21,10 +21,4 @@
     </link>
     <link name="${name}box_link" >
-      <collision>
-        <origin xyz="0 0 0.0325" rpy="0 0 0"/>
-        <geometry>
-          <box size="0.07 0.085 0.065"/>
-        </geometry>
-      </collision>
       <visual>
         <origin xyz="0 0 0" rpy="0 0 0" />
@@ -36,18 +30,12 @@
      <inertial>
        <origin xyz="0 0 ${base_to_box_height/2}" rpy="0 0 0"/>
-       <mass value="1"/>
+       <mass value="0.28"/>
        <inertia
-	    ixx="1.0" ixy="0.0" ixz="0.0"
-	    iyy="1.0" iyz="0.0"
-	    izz="1.0"/>
+	    ixx="0.00190" ixy="0.0" ixz="0.0"
+	    iyy="0.00202" iyz="0.0"
+	    izz="0.00152"/>
      </inertial>
     </link>
     <link name="${name}plate_link">
-      <collision>
-        <origin xyz="0 0 0.0015" rpy="0 0 0"/>
-        <geometry>
-          <box size="0.35 0.095 0.003"/>
-        </geometry>
-      </collision>
       <visual>
         <origin xyz="-0.075 0 0" rpy="0 0 0" />
@@ -59,18 +47,12 @@
      <inertial>
        <origin xyz="0 0 0.0015" rpy="0 0 0"/>
-       <mass value="1"/>
+       <mass value="0.08"/>
        <inertia
-	    ixx="1.0" ixy="0.0" ixz="0.0"
-	    iyy="1.0" iyz="0.0"
-	    izz="1.0"/>
+	    ixx="0.00150" ixy="0.0" ixz="0.0"
+	    iyy="0.02191" iyz="0.0"
+	    izz="0.02041"/>
      </inertial>
     </link>
     <link name="left_pt_pillars" >
-      <collision>
-        <origin xyz="0 0 0.10" rpy="0 0 0"/>
-        <geometry>
-          <box size="0.01 0.05 0.20"/>
-        </geometry>
-      </collision>
       <visual>
         <origin xyz="0 0 0" rpy="0 0 0" />
@@ -82,18 +64,12 @@
      <inertial>
        <origin xyz="0 0 0.01" rpy="0 0 0"/>
-       <mass value="1"/>
+       <mass value="0.06"/>
        <inertia
-	    ixx="1.0" ixy="0.0" ixz="0.0"
-	    iyy="1.0" iyz="0.0"
-	    izz="1.0"/>
+	    ixx="0.00708" ixy="0.0" ixz="0.0"
+	    iyy="0.00043" iyz="0.0"
+	    izz="0.00668"/>
      </inertial>
     </link>
     <link name="right_pt_pillars" >
-      <collision>
-        <origin xyz="0 0 0.10" rpy="0 0 0"/>
-        <geometry>
-          <box size="0.01 0.05 0.20"/>
-        </geometry>
-      </collision>
       <visual>
         <origin xyz="0 0 0" rpy="0 0 0" />
@@ -105,5 +81,5 @@
      <inertial>
        <origin xyz="0 0 0.01" rpy="0 0 0"/>
-       <mass value="1"/>
+       <mass value="0.06"/>
        <inertia
 	    ixx="1.0" ixy="0.0" ixz="0.0"
@@ -113,10 +89,4 @@
     </link>
     <link name="${name}projector_link">
-      <collision>
-        <origin xyz="0 0 0.035" rpy="0 0 0"/>
-        <geometry>
-          <box size="0.24 0.17 0.07"/>
-        </geometry>
-      </collision>
       <visual>
         <origin xyz="0.07 0.037 0" rpy="0 0 0" />
@@ -128,9 +98,9 @@
      <inertial>
        <origin xyz="0 0 0.035" rpy="0 0 0"/>
-       <mass value="1"/>
+       <mass value="2"/>
        <inertia
-	    ixx="1.0" ixy="0.0" ixz="0.0"
-	    iyy="1.0" iyz="0.0"
-	    izz="1.0"/>
+	    ixx="0.00536" ixy="0.0" ixz="0.0"
+	    iyy="0.01441" iyz="0.0"
+	    izz="0.01041"/>
      </inertial>
     </link>

Commit message: fix pan and tilt joint effort

File: urdf/pantilt/pantilt.urdf.xacro (robot description, xacro)
@@ -116,5 +116,6 @@
       <origin xyz="0 0 ${base_to_box_height/2}" rpy="0 0 0" />
       <axis xyz="0 0 1" />
-      <limit lower="0" upper="2" effort="1" velocity="1"/>
+      <limit lower="0" upper="2" effort="41" velocity="1"/>
+      <!--<safety_controller k_velocity="10" k_position="15" soft_lower_limit="-2.0" soft_upper_limit="0.5" />-->
       <dynamics damping="0.7"/>
     </joint>
@@ -134,5 +135,6 @@
       <origin xyz="0 0 ${box_to_proj_height}" rpy="0 0 3.14" />
       <axis xyz="1 0 0" />
-      <limit lower="0" upper="2" effort="1" velocity="1"/>
+      <limit lower="0" upper="2" effort="10" velocity="1"/>
+      <!--<safety_controller k_velocity="10" k_position="15" soft_lower_limit="-2.0" soft_upper_limit="0.5" />-->
       <dynamics damping="0.7"/>
     </joint>

Commit message: [Fix] Pan and Tilt joint limit

File: urdf/pantilt/pantilt.urdf.xacro (robot description, xacro)
@@ -116,5 +116,5 @@
       <origin xyz="0 0 ${base_to_box_height/2}" rpy="0 0 0" />
       <axis xyz="0 0 1" />
-      <limit lower="0" upper="2" effort="41" velocity="1"/>
+      <limit lower="-2.9670" upper="2.9670" effort="41" velocity="1"/>
       <!--<safety_controller k_velocity="10" k_position="15" soft_lower_limit="-2.0" soft_upper_limit="0.5" />-->
       <dynamics damping="0.7"/>
@@ -135,5 +135,5 @@
       <origin xyz="0 0 ${box_to_proj_height}" rpy="0 0 3.14" />
       <axis xyz="1 0 0" />
-      <limit lower="0" upper="2" effort="10" velocity="1"/>
+      <limit lower="-0.2617" upper="0.7853" effort="10" velocity="1"/>
       <!--<safety_controller k_velocity="10" k_position="15" soft_lower_limit="-2.0" soft_upper_limit="0.5" />-->
       <dynamics damping="0.7"/>

Commit message: [Fix] tilt joint limit

File: urdf/pantilt/pantilt.urdf.xacro (robot description, xacro)
@@ -135,5 +135,5 @@
       <origin xyz="0 0 ${box_to_proj_height}" rpy="0 0 3.14" />
       <axis xyz="1 0 0" />
-      <limit lower="-0.2617" upper="0.7853" effort="10" velocity="1"/>
+      <limit lower="-0.2617" upper="1.3" effort="10" velocity="1"/>
       <!--<safety_controller k_velocity="10" k_position="15" soft_lower_limit="-2.0" soft_upper_limit="0.5" />-->
       <dynamics damping="0.7"/>

Commit message: [Add] ud_pt_projector_optical_frame

File: urdf/pantilt/pantilt.urdf.xacro (robot description, xacro)
@@ -105,4 +105,5 @@
      </inertial>
     </link>
+    <link name="${name}projector_optical_frame"/>
     <joint name="${name}base_joint" type="fixed">
       <parent link="${name}base_link"/>
@@ -120,10 +121,10 @@
       <dynamics damping="0.7"/>
     </joint>
-    <joint name="ud_pt_plate_link_to_left_pt_pillars" type="fixed">
+    <joint name="${name}plate_link_to_left_pt_pillars" type="fixed">
       <parent link="${name}plate_link"/>
       <child link="left_pt_pillars"/>
       <origin xyz="0.09 0 0.1" rpy="0 0 0" />
     </joint>
-    <joint name="ud_pt_plate_link_to_right_pt_pillars" type="fixed">
+    <joint name="${name}plate_link_to_right_pt_pillars" type="fixed">
       <parent link="${name}plate_link"/>
       <child link="right_pt_pillars"/>
@@ -139,4 +140,9 @@
       <dynamics damping="0.7"/>
     </joint>
+    <joint name="${name}projector_link_to_${name}projector_optical_frame" type="fixed">
+      <parent link="${name}projector_link"/>
+      <child link="${name}projector_optical_frame"/>
+      <origin xyz="0 -0.02 0" rpy="0 0 3.14" />
+    </joint>
   </xacro:macro>
   <xacro:pantilt_name name="ud_pt_"/>

Commit message: [Change pantilt.urdf.xacro]

File: urdf/pantilt/pantilt.urdf.xacro (robot description, xacro)
@@ -143,5 +143,5 @@
       <parent link="${name}projector_link"/>
       <child link="${name}projector_optical_frame"/>
-      <origin xyz="0 -0.02 0" rpy="0 0 3.14" />
+      <origin xyz="0 -0.02 0" rpy="-1.56 0 3.14" />
     </joint>
   </xacro:macro>

Commit message: [Add] pantilt dae files

File: urdf/pantilt/pantilt.urdf.xacro (robot description, xacro)
@@ -23,5 +23,5 @@
         <geometry>
           <!--box size="0.07 0.085 0.065" /-->
-          <mesh filename="package://ubiquitous_display_description/meshes/STL/ud_pt_base.stl" scale="0.001 0.001 0.001"/>
+          <mesh filename="package://ubiquitous_display_description/meshes/DAE/ud_pt_base.dae" scale="0.001 0.001 0.001"/>
         </geometry>
         <material name="gray"/>
@@ -41,5 +41,5 @@
         <geometry>
           <!--box size="0.35 0.095 0.003" /-->
-          <mesh filename="package://ubiquitous_display_description/meshes/STL/ud_pt_pan.stl" scale="0.001 0.001 0.001"/>
+          <mesh filename="package://ubiquitous_display_description/meshes/DAE/ud_pt_pan.dae" scale="0.001 0.001 0.001"/>
         </geometry>
         <material name="gray"/>
@@ -59,5 +59,5 @@
         <geometry>
           <!--box size="0.24 0.17 0.07" /-->
-          <mesh filename="package://ubiquitous_display_description/meshes/STL/ud_pt_tilt.stl" scale="0.001 0.001 0.001"/>
+          <mesh filename="package://ubiquitous_display_description/meshes/DAE/ud_pt_tilt.dae" scale="0.001 0.001 0.001"/>
         </geometry>
         <material name="gray"/>

Commit message: [Fix] dae name

File: urdf/pantilt/pantilt.urdf.xacro (robot description, xacro)
@@ -23,5 +23,5 @@
         <geometry>
           <!--box size="0.07 0.085 0.065" /-->
-          <mesh filename="package://ubiquitous_display_description/meshes/DAE/ud_pt_base.dae" scale="0.001 0.001 0.001"/>
+          <mesh filename="package://ubiquitous_display_description/meshes/DAE/pantilt_base.dae" scale="0.001 0.001 0.001"/>
         </geometry>
         <material name="gray"/>
@@ -41,5 +41,5 @@
         <geometry>
           <!--box size="0.35 0.095 0.003" /-->
-          <mesh filename="package://ubiquitous_display_description/meshes/DAE/ud_pt_pan.dae" scale="0.001 0.001 0.001"/>
+          <mesh filename="package://ubiquitous_display_description/meshes/DAE/pan_link.dae" scale="0.001 0.001 0.001"/>
         </geometry>
         <material name="gray"/>
@@ -59,5 +59,5 @@
         <geometry>
           <!--box size="0.24 0.17 0.07" /-->
-          <mesh filename="package://ubiquitous_display_description/meshes/DAE/ud_pt_tilt.dae" scale="0.001 0.001 0.001"/>
+          <mesh filename="package://ubiquitous_display_description/meshes/DAE/tilt_link.dae" scale="0.001 0.001 0.001"/>
         </geometry>
         <material name="gray"/>
@@ -77,5 +77,5 @@
         <geometry>
           <!--box size="0.24 0.17 0.07" /-->
-          <mesh filename="package://ubiquitous_display_description/meshes/STL/projector.stl" scale="0.001 0.001 0.001"/>
+          <mesh filename="package://ubiquitous_display_description/meshes/DAE/projector.dae" scale="0.001 0.001 0.001"/>
         </geometry>
         <material name="gray"/>

Commit message: [Edit] joint (projector_link and projector_optical_frame

File: urdf/pantilt/pantilt.urdf.xacro (robot description, xacro)
@@ -121,5 +121,5 @@
     </joint>
     <joint name="projector_link_to_projector_optical_frame" type="fixed">
-      <origin xyz="0 0.0805 0 " rpy="-1.57 0 0" />
+      <origin xyz="0 0 0 " rpy="-1.57 0 0" />
       <parent link="projector_link"/>
       <child link="projector_optical_frame"/>
