Commit message: fixed

File: urdf/youbot/base.urdf.xacro (robot description, xacro)
@@ -56,5 +56,5 @@
         <geometry>
           <!--<box size="${base_size_x} ${base_size_y} ${base_size_z}" />-->
-          <mesh filename="package://ubiquitous_display_description/meshes/DAE/base_convex.dae"/>
+          <mesh filename="package://ubiquitous_display_description/meshes/DAE/sbase_convex.dae"/>
         </geometry>
       </collision>

Commit message: fixed typo

File: urdf/youbot/base.urdf.xacro (robot description, xacro)
@@ -56,5 +56,5 @@
         <geometry>
           <!--<box size="${base_size_x} ${base_size_y} ${base_size_z}" />-->
-          <mesh filename="package://ubiquitous_display_description/meshes/DAE/sbase_convex.dae"/>
+          <mesh filename="package://ubiquitous_display_description/meshes/DAE/base_convex.dae"/>
         </geometry>
       </collision>

Commit message: replace base.urdf.xacro

File: urdf/youbot/base.urdf.xacro (robot description, xacro)
@@ -5,6 +5,6 @@
        xmlns:xacro="http://ros.org/wiki/xacro">
   <!-- sensors -->
-  <xacro:include filename="$(find ubiquitous_display_description)/urdf/youbot/base.gazebo.xacro"/>
-  <xacro:include filename="$(find ubiquitous_display_description)/urdf/youbot/base.transmission.xacro"/>
+  <xacro:include filename="$(find youbot_description)/urdf/youbot_base/base.gazebo.xacro"/>
+  <xacro:include filename="$(find youbot_description)/urdf/youbot_base/base.transmission.xacro"/>
   <!-- simplified box collision geometry for base -->
   <xacro:property name="base_size_x" value="0.570"/>
@@ -33,9 +33,28 @@
   <xacro:property name="wheel_joint_safety_k_velocity" value="10.0"/>
   <xacro:macro name="youbot_base" params="name">
-    <link name="${name}_footprint"/>
+    <link name="${name}_footprint">
+      <inertial>
+        <mass value="0.1"/>
+        <origin xyz="0 0 ${-base_size_z / 2.0}" rpy="0 0 0"/>
+        <inertia ixx="1.0" ixy="0.0" ixz="0.0" iyy="1.0" iyz="0.0" izz="1.0"/>
+      </inertial>
+      <visual>
+        <origin xyz="0 0 0" rpy="0 0 0"/>
+        <geometry>
+          <box size="0.001 0.001 0.001"/>
+        </geometry>
+        <material name="Red"/>
+      </visual>
+      <collision>
+        <origin xyz="0 0 ${-base_size_z / 2.0}" rpy="0 0 0"/>
+        <geometry>
+          <box size="0.001 0.001 0.001"/>
+        </geometry>
+      </collision>
+    </link>
     <joint name="${name}_footprint_joint" type="fixed">
-      <origin xyz="0 0 0.10" rpy="0 0 0"/>
+      <origin xyz="0 0 0" rpy="0 0 0"/>
+      <child link="${name}_link"/>
       <parent link="${name}_footprint"/>
-      <child link="${name}_link"/>
     </joint>
     <link name="${name}_link">
@@ -48,5 +67,5 @@
         <origin xyz="0 0 0" rpy="0 0 0"/>
         <geometry>
-          <mesh filename="package://ubiquitous_display_description/meshes/DAE/base.dae"/>
+          <mesh filename="package://youbot_description/meshes/youbot_base/base.dae"/>
         </geometry>
         <material name="DarkGrey"/>
@@ -56,5 +75,5 @@
         <geometry>
           <!--<box size="${base_size_x} ${base_size_y} ${base_size_z}" />-->
-          <mesh filename="package://ubiquitous_display_description/meshes/DAE/base_convex.dae"/>
+          <mesh filename="package://youbot_description/meshes/youbot_base/base_convex.dae"/>
         </geometry>
       </collision>

Commit message: [Change] youbot DAE file directory

File: urdf/youbot/base.urdf.xacro (robot description, xacro)
@@ -64,5 +64,5 @@
         <origin xyz="0 0 0" rpy="0 0 0"/>
         <geometry>
-          <mesh filename="package://youbot_description/meshes/youbot_base/base.dae"/>
+          <mesh filename="package://ubiquitous_display_description/meshes/DAE/base.dae"/>
         </geometry>
         <material name="DarkGrey"/>
@@ -72,5 +72,5 @@
         <geometry>
           <!--<box size="${base_size_x} ${base_size_y} ${base_size_z}" />-->
-          <mesh filename="package://youbot_description/meshes/youbot_base/base_convex.dae"/>
+          <mesh filename="package://ubiquitous_display_description/meshes/DAE/base_convex.dae"/>
         </geometry>
       </collision>

Commit message: [Fix] base_joint z pose

File: urdf/youbot/base.urdf.xacro (robot description, xacro)
@@ -51,5 +51,5 @@
     </link>
     <joint name="${name}_footprint_joint" type="fixed">
-      <origin xyz="0 0 0.08" rpy="0 0 0"/>
+      <origin xyz="0 0 0.03" rpy="0 0 0"/>
       <child link="${name}_link"/>
       <parent link="${name}_footprint"/>
