Commit message: [Republish] ubiquitous_display.urdf

File: robots/ubiquitous_display.urdf (robot description, URDF)
Before this commit: robot ubiquitous_didsplay, 29 links, 28 joints
Links:
- link front_laser_frame: geometry collision box size=0.058 0.058 0.087; visual mesh filename=package://ubiquitous_display_description/meshes/DAE/hokuyo_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
- link kinect2_rgb_optical_frame: mass None -> 0.2; geometry collision box size=0.25 0.065 0.068; visual mesh filename=package://ubiquitous_display_description/meshes/STL/kinect2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 scale=0.001 0.001 0.001
- link left_pt_pillars: mass None -> 0.06
- link rear_laser_frame: geometry collision box size=0.058 0.058 0.087; visual mesh filename=package://ubiquitous_display_description/meshes/DAE/hokuyo_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
- link right_pt_pillars: mass None -> 0.06
- link ud_base_footprint: mass None -> 0.1; geometry collision box size=0.001 0.001 0.001; visual box size=0.001 0.001 0.001
- link ud_base_link: geometry collision mesh filename=package://youbot_description/meshes/youbot_base/base_convex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; visual mesh filename=package://youbot_description/meshes/youbot_base/base.dae
- link ud_pt_box_link: mass None -> 0.28
- link ud_pt_plate_link: mass None -> 0.08
- link ud_pt_projector_link: mass None -> 2
Joints:
- joint pan_joint: limit lower=0 upper=2 effort=1 velocity=1 -> lower=-2.9670 upper=2.9670 effort=41 velocity=1
- joint tilt_joint: limit lower=0 upper=2 effort=1 velocity=1 -> lower=-0.2617 upper=0.7853 effort=10 velocity=1
- joint ud_base_footprint_joint: origin xyz=0 0 0.10 rpy=0 0 0 -> xyz=0 0 0 rpy=0 0 0

Commit message: recreate ud.urdf

File: robots/ubiquitous_display.urdf (robot description, URDF)
Before this commit: robot ubiquitous_display, 29 links, 28 joints
Links:
- link front_laser_adjuster_link: geometry visual box size=0.18 0.02 0.02
- link rear_laser_adjuster_link: geometry visual box size=0.18 0.02 0.02

Commit message: [Add] body.gazebo.xacro

File: robots/ubiquitous_display.urdf (robot description, URDF)
Before this commit: robot ubiquitous_display, 29 links, 28 joints
Links:
- added link ud_pt_projector_optical_frame
- link ud_base_link: geometry collision mesh filename=package://ubiquitous_display_description/meshes/DAE/base_co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; visual mesh filename=package://ubiquitous_display_description/meshes/DAE/base.dae
Joints:
- added joint ud_pt_projector_link_to_ud_pt_projector_optical_frame: type fixed, parent ud_pt_projector_link, child ud_pt_projector_optical_frame, origin xyz=0 -0.02 0 rpy=-1.56 0 3.14
- joint kinect2_plate_to_kinect2_rgb_optical_frame: origin xyz=0.095 0 0.035  rpy=0 0 0 -> xyz=0.095 0 0.035  rpy=-1.56 0 0
- joint tilt_joint: limit lower=-0.2617 upper=0.7853 effort=10 velocity=1 -> lower=-0.2617 upper=1.3 effort=10 velocity=1; origin xyz=0 0 0.17 rpy=0 0 3.14 -> xyz=0 0 0.17 rpy=0 0 0
- joint top_plate_link_to_ud_pt_base_link: origin xyz=0 0 0.0325  rpy=0 0 0 -> xyz=0 0 0.0325  rpy=0 0 3.14
- joint ud_pt_plate_link_to_left_pt_pillars: origin xyz=0.09 0 0.1 rpy=0 0 0 -> xyz=-0.09 0 0.1 rpy=0 0 0
- joint ud_pt_plate_link_to_right_pt_pillars: origin xyz=-0.24 0 0.1 rpy=0 0 0 -> xyz=0.24 0 0.1 rpy=0 0 0

File: urdf/body/body.urdf.xacro (robot description, xacro)
@@ -1,4 +1,5 @@
 <?xml version="1.0"?>
 <robot name="body" xmlns:xacro="http://www.ros.org/wiki/xacro">
+  <xacro:include filename="$(find ubiquitous_display_description)/urdf/body/body.gazebo.xacro"/>
   <!-- Definition of various sizes -->
   <xacro:property name="bottom_pillar_height" value="0.1"/>
@@ -53,5 +54,7 @@
       <xacro:pillar_template height="${pillar_height}" origin_x="${-pillar_offset_x}" origin_y="${-pillar_offset_y}"/>
     </link>
+    <xacro:pillar_template_gazebo name="${name}"/>
     <xacro:plate_template name="${name}"/>
+    <xacro:plate_template_gazebo name="${name}"/>
     <joint name="${name}_pillars_to_${name}_plate_joint" type="fixed">
       <parent link="${name}_pillars_link"/>
@@ -89,4 +92,5 @@
   <!-- Front -->
   <xacro:laser_adjuster_template name="front"/>
+  <xacro:laser_adjuster_template_gazebo name="front"/>
   <joint name="front_laser_adjuster_joint" type="fixed">
     <origin xyz="${adjuster_offset_x} 0 0" rpy="0 0 0"/>
@@ -96,4 +100,5 @@
   <!-- Rear -->
   <xacro:laser_adjuster_template name="rear"/>
+  <xacro:laser_adjuster_template_gazebo name="rear"/>
   <joint name="rear_laser_adjuster_joint" type="fixed">
   <origin xyz="${-adjuster_offset_x} 0 0" rpy="0 0 3.1415"/>

File: urdf/sensor/kinect/kinect2.urdf.xacro (robot description, xacro)
@@ -28,5 +28,5 @@
       </collision>
       <visual>
-        <origin rpy="-1.56 0 0" xyz="0 0 0"/>
+        <origin rpy="0 0 0" xyz="0 0 0"/>
         <geometry>
             <!-- these meshes were exported in mm, so scale back to m -->
@@ -47,5 +47,5 @@
     <link name="kinect2_ir_optical_frame">
       <visual>
-        <origin rpy="0.075 0 0" xyz="0 0 0"/>
+        <origin rpy="0 0 0" xyz="0 0 0"/>
         <geometry>
           <sphere radius="0.0005"/>

Commit message: [Fix] pantilt xacro name and [Add] kinect2 parent argument

File: robots/ubiquitous_display.urdf (robot description, URDF)
Before this commit: robot ubiquitous_display, 30 links, 29 joints
Links:
- removed link ud_base_footprint
- removed link ud_base_link
- added link base_footprint, mass 0.1; collision box size=0.001 0.001 0.001; visual box size=0.001 0.001 0.001
- added link base_link, mass 22.0; collision mesh filename=package://ubiquitous_display_description/meshes/DAE/base_co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; visual mesh filename=package://ubiquitous_display_description/meshes/DAE/base.dae
- link bottom_pillars_link: geometry visual cylinder length=0.14 radius=0.01; visual cylinder length=0.14 radius=0.01
Joints:
- removed joint ud_base_footprint_joint
- removed joint ud_base_link_to_bottom_pillars_link
- added joint base_footprint_joint: type fixed, parent base_footprint, child base_link, origin xyz=0 0 0.08 rpy=0 0 0
- added joint base_link_to_bottom_pillars_link: type fixed, parent base_link, child bottom_pillars_link, origin xyz=0 0 0 rpy=0 0 0
- joint bottom_pillars_to_bottom_plate_joint: origin xyz=0 0 0.1 -> xyz=0 0 0.14
- joint caster_joint_bl: parent ud_base_link -> base_link
- joint caster_joint_br: parent ud_base_link -> base_link
- joint caster_joint_fl: parent ud_base_link -> base_link
- joint caster_joint_fr: parent ud_base_link -> base_link

File: robots/ubiquitous_display.urdf.xacro (robot description, xacro)
@@ -6,8 +6,8 @@
   <xacro:include filename="$(find ubiquitous_display_description)/urdf/youbot/youbot_base_only.urdf.xacro"/>
   <xacro:include filename="$(find ubiquitous_display_description)/urdf/sensor/lrf/hokuyo_utm30lx.urdf.xacro"/>
-  <xacro:pantilt_name name="ud_pt_" parent="top_plate_link"/>
+  <xacro:pantilt_model name="ud_pt_" parent="top_plate_link"/>
   <xacro:hokuyo_utm30lx_model name="front_laser" parent="front_laser_adjuster_link" />
   <xacro:hokuyo_utm30lx_model name="rear_laser" parent="rear_laser_adjuster_link" />
-  <xacro:kinect2_model name="ud_pt_"/>
+  <xacro:kinect2_model name="ud_pt_" parent="kinect2_plate_link"/>
   <!-- =============== Gazebo =============== -->
   <gazebo>

File: urdf/pantilt/pantilt.urdf.xacro (robot description, xacro)
@@ -17,5 +17,5 @@
     <color rgba="0.7 0.7 0.7 1.0" />
   </material>
-  <xacro:macro name="pantilt_name" params="name parent">
+  <xacro:macro name="pantilt_model" params="name parent">
     <link name="${name}base_link" >
     </link>

File: urdf/sensor/kinect/kinect2.urdf.xacro (robot description, xacro)
@@ -5,5 +5,5 @@
 <robot xmlns:xacro="http://www.ros.org/wiki/xacro" name="kinect2">
   <xacro:include filename="$(find ubiquitous_display_description)/urdf/sensor/kinect/kinect2.gazebo.xacro"/>
-  <xacro:macro name="kinect2_model" params="name">
+  <xacro:macro name="kinect2_model" params="name parent">
     <link name="kinect2_plate_link">
       <visual>
@@ -18,5 +18,5 @@
       <origin xyz="0.075 -0.11 0.135" rpy="0 0 3.14" />
       <parent link="${name}projector_link" />
-      <child link="kinect2_plate_link" />
+      <child link="${parent}" />
     </joint>
     <link name="kinect2_rgb_optical_frame">

Commit message: [Fix] frame link name in base_controller(youbot.gazebo.xacro)

File: robots/ubiquitous_display.urdf (robot description, URDF)
Before this commit: robot ubiquitous_display, 30 links, 29 joints
Links:
- added link camera_ir_optical_frame; visual sphere radius=0.0005
- added link camera_rgb_optical_frame; visual sphere radius=0.0005
Joints:
- added joint kinect2_ir_optical_frame_to_camera_ir_optical_frame: type fixed, parent kinect2_ir_optical_frame, child camera_ir_optical_frame, origin xyz=0 0 0  rpy=1.56 0 0
- added joint kinect2_rgb_optical_frame_to_camera_rgb_optical_frame: type fixed, parent kinect2_rgb_optical_frame, child camera_rgb_optical_frame, origin xyz=0 0 0  rpy=1.56 0 0

File: urdf/youbot/base.gazebo.xacro (robot description, xacro)
@@ -51,5 +51,5 @@
         <odometryFrame>odom</odometryFrame>
         <odometryRate>100.0</odometryRate>
-        <robotBaseFrame>ud_base_footprint</robotBaseFrame>
+        <robotBaseFrame>base_footprint</robotBaseFrame>
       </plugin>
     </gazebo>

Commit message: [Fix] kinect coordination

File: robots/ubiquitous_display.urdf (robot description, URDF)
Before this commit: robot ubiquitous_display, 32 links, 31 joints
Joints:
- joint kinect2_ir_optical_frame_to_camera_ir_optical_frame: origin xyz=0 0 0  rpy=1.56 0 0 -> xyz=0 0 0  rpy=-1.56 0 -1.56
- joint kinect2_rgb_optical_frame_to_camera_rgb_optical_frame: origin xyz=0 0 0  rpy=1.56 0 0 -> xyz=0 0 0  rpy=-1.56 0 -1.56

File: urdf/sensor/kinect/kinect2.gazebo.xacro (robot description, xacro)
@@ -22,5 +22,5 @@
           <alwaysOn>true</alwaysOn>
           <updateRate>1.0</updateRate>
-          <cameraName>${camera_name}_ir</cameraName>
+          <cameraName>${camera_name}</cameraName>
           <imageTopicName>/${camera_name}/depth/image_raw</imageTopicName>
           <cameraInfoTopicName>/${camera_name}/depth/camera_info</cameraInfoTopicName>
@@ -42,5 +42,5 @@
         </plugin>
       </sensor>
-      <material value="Gazebo/Black"/>
+      <!--material>Gazebo/Black</material-->
     </gazebo>
   </xacro:macro>
@@ -65,10 +65,10 @@
 					<alwaysOn>true</alwaysOn>
 					<updateRate>1.0</updateRate>
-					<cameraName>${camera_name}_rgb</cameraName>
+					<cameraName>${camera_name}</cameraName>
 					<imageTopicName>/${camera_name}/rgb/image_raw</imageTopicName>
 					<cameraInfoTopicName>/${camera_name}/rgb/camera_info</cameraInfoTopicName>
-					<depthImageTopicName>/${camera_name}/depth/image_raw</depthImageTopicName>
-					<depthImageCameraInfoTopicName>/${camera_name}/depth/camera_info</depthImageCameraInfoTopicName>
-					<pointCloudTopicName>/${camera_name}/depth_registered/points</pointCloudTopicName>
+					<depthImageTopicName>/${camera_name}/rgb/image_raw</depthImageTopicName>
+					<depthImageCameraInfoTopicName>/${camera_name}/rgb/camera_info</depthImageCameraInfoTopicName>
+					<pointCloudTopicName>/${camera_name}/rgb/points</pointCloudTopicName>
 					<frameName>${frame_name}</frameName>
 					<pointCloudCutoff>0.5</pointCloudCutoff>
@@ -85,5 +85,5 @@
 				</plugin>
 			</sensor>
-			<material value="Gazebo/Black"/>
+			<!--material>Gazebo/Black</material-->
 		</gazebo>
 	</xacro:macro>

File: urdf/sensor/kinect/kinect2.urdf.xacro (robot description, xacro)
@@ -63,4 +63,7 @@
       <child link="kinect2_ir_optical_frame"/>
     </joint>
+    <gazebo reference="kinect2_rgb_optical_frame">
+      <material>Gazebo/Black</material>
+    </gazebo>
   </xacro:macro>
 </robot>

File: urdf/sensor/kinect/kinect2_for_gazebo.urdf.xacro (robot description, xacro)
@@ -25,16 +25,16 @@
     </link>
     <joint name="kinect2_rgb_optical_frame_to_${name}_rgb_optical_frame" type="fixed">
-      <origin xyz="0 0 0 " rpy="1.56 0 0" />
+      <origin xyz="0 0 0.05 " rpy="1.57 -1.57 -1.57" />
       <parent link="${rgb_parent}"/>
       <child link="${name}_rgb_optical_frame"/>
     </joint>
     <joint name="kinect2_ir_optical_frame_to_${name}_ir_optical_frame" type="fixed">
-      <origin xyz="0 0 0 " rpy="1.56 0 0" />
+      <origin xyz="0 0 0.05 " rpy="-1.57 -1.57 -1.57" />
       <parent link="${depth_parent}"/>
       <child link="${name}_ir_optical_frame"/>
     </joint>
     <!--<xacro:camera_gazebo link_name="kinect2_rgb" frame_name="kinect2_rgb_optical_frame"/>-->
-    <xacro:kinect_ir_sensor_gazebo link_name="${name}_ir" frame_name="${name}_ir_optical_frame" camera_name="${name}" />
-    <xacro:kinect_rgb_sensor_gazebo link_name="${name}_rgb" frame_name="${name}_rgb_optical_frame" camera_name="${name}" />
+    <xacro:kinect_ir_sensor_gazebo link_name="${name}_ir" frame_name="${name}_ir_optical_frame" camera_name="${name}_ir" />
+    <xacro:kinect_rgb_sensor_gazebo link_name="${name}_rgb" frame_name="${name}_rgb_optical_frame" camera_name="${name}_rgb" />
   </xacro:macro>
 </robot>
