Commit message: [Add] kinect2_for_gazebo.urdf.xacro

File: robots/ubiquitous_display_for_gazebo.urdf.xacro (robot description, xacro)
@@ -3,5 +3,4 @@
   <xacro:include filename="$(find ubiquitous_display_description)/urdf/body/body.urdf.xacro"/>
   <xacro:include filename="$(find ubiquitous_display_description)/urdf/pantilt/pantilt.urdf.xacro"/>
-  <xacro:include filename="$(find ubiquitous_display_description)/urdf/sensor/kinect/kinect2.urdf.xacro"/>
   <xacro:include filename="$(find ubiquitous_display_description)/urdf/youbot/youbot_base_only.urdf.xacro"/>
   <xacro:include filename="$(find ubiquitous_display_description)/urdf/sensor/lrf/hokuyo_utm30lx.urdf.xacro"/>
@@ -10,6 +9,5 @@
   <xacro:hokuyo_utm30lx_model name="front_laser" parent="front_laser_adjuster_link" />
   <xacro:hokuyo_utm30lx_model name="rear_laser" parent="rear_laser_adjuster_link" />
-  <xacro:kinect2_model name="ud_pt_" parent="kinect2_plate_link"/>
-  <xacro:kinect2_for_gazebo_model name="camera" rgb_parent="kinect2_rgb_optical_frame" depth_parent="kinect2_ir_optical_frame"/>
+  <!--xacro:kinect2_for_gazebo_model name="ud_pt_" camera_name="camera"/-->
   <!-- =============== Gazebo =============== -->
   <gazebo>

File: urdf/sensor/kinect/kinect2.urdf.xacro (robot description, xacro)
@@ -56,7 +56,4 @@
       <child link="kinect2_ir_optical_frame"/>
     </joint>
-    <gazebo reference="kinect2_rgb_optical_frame">
-      <material>Gazebo/Black</material>
-    </gazebo>
   </xacro:macro>
 </robot>

File: urdf/sensor/kinect/kinect2_for_gazebo.urdf.xacro (robot description, xacro)
@@ -5,36 +5,59 @@
 <robot xmlns:xacro="http://www.ros.org/wiki/xacro" name="kinect2_for_gazebo">
   <xacro:include filename="$(find ubiquitous_display_description)/urdf/sensor/kinect/kinect2.gazebo.xacro"/>
-  <xacro:macro name="kinect2_for_gazebo_model" params="name rgb_parent depth_parent">
-    <link name="${name}_rgb_optical_frame">
+  <xacro:macro name="kinect2_for_gazebo_model" params="name camera_name">
+    <link name="${camera_name}_plate_link">
       <visual>
-        <origin rpy="0 0 0" xyz="0 0 0"/>
+        <origin xyz="0 0 0" rpy="0 0 0" />
         <geometry>
-          <sphere radius="0.0005"/>
+          <box size="0.25 0.015 0.01" />
+        </geometry>
+        <material name="gray"/>
+      </visual>
+    </link>
+    <joint name="${name}projector_link_to_${camera_name}_plate_link" type="fixed">
+      <origin xyz="0.075 -0.11 0.135" rpy="0 0 3.14" />
+      <parent link="${name}projector_link" />
+      <child link="${camera_name}_plate_link" />
+    </joint>
+    <link name="${camera_name}_rgb_optical_frame">
+      <collision>
+        <origin xyz="-1.56 0 0" rpy="0 0 0"/>
+        <geometry>
+          <box size="0.25 0.065 0.068"/>
+        </geometry>
+      </collision>
+      <visual>
+        <origin rpy="-1.56 0 0" xyz="0 0 0"/>
+        <geometry>
+            <!-- these meshes were exported in mm, so scale back to m -->
+          <mesh filename="package://ubiquitous_display_description/meshes/STL/kinect2_origin_on_rgb_optical_frame.stl" scale="0.001 0.001 0.001"/>
+          <!--box size="0.25 0.07 0.6" /-->
         </geometry>
         <material name="black"/>
       </visual>
+      <inertial>
+        <mass value="0.2" />
+        <origin xyz="-1.56 0 0" rpy="0 0 0"/>
+        <inertia
+          ixx="0.00147" ixy="0" ixz="0"
+          iyy="0.01112" iyz="0"
+          izz="0.01118" />
+      </inertial>
     </link>
-    <link name="${name}_ir_optical_frame">
-      <visual>
-        <origin rpy="0 0 0" xyz="0 0 0"/>
-        <geometry>
-          <sphere radius="0.0005"/>
-        </geometry>
-        <material name="black"/>
-      </visual>
+    <link name="${camera_name}_ir_optical_frame">
     </link>
-    <joint name="kinect2_rgb_optical_frame_to_${name}_rgb_optical_frame" type="fixed">
-      <origin xyz="0 0 0.05 " rpy="1.57 -1.57 -1.57" />
-      <parent link="${rgb_parent}"/>
-      <child link="${name}_rgb_optical_frame"/>
+    <joint name="${camera_name}_plate_to_${camera_name}_rgb_optical_frame" type="fixed">
+      <origin xyz="0.095 0 0.08 " rpy="0 -1.57 -1.57" />
+      <parent link="${camera_name}_plate_link"/>
+      <child link="${camera_name}_rgb_optical_frame"/>
     </joint>
-    <joint name="kinect2_ir_optical_frame_to_${name}_ir_optical_frame" type="fixed">
-      <origin xyz="0 0 0.05 " rpy="-1.57 -1.57 -1.57" />
-      <parent link="${depth_parent}"/>
-      <child link="${name}_ir_optical_frame"/>
+    <joint name="${camera_name}_rgb_optical_frame_to_${camera_name}_ir_optical_frame" type="fixed">
+      <origin xyz="-0.0425 0 0.045 " rpy="-1.57 -1.57 -1.57" />
+      <parent link="${camera_name}_rgb_optical_frame"/>
+      <child link="${camera_name}_ir_optical_frame"/>
     </joint>
     <!--<xacro:camera_gazebo link_name="kinect2_rgb" frame_name="kinect2_rgb_optical_frame"/>-->
-    <xacro:kinect_ir_sensor_gazebo link_name="${name}_ir" frame_name="${name}_ir_optical_frame" camera_name="${name}_ir" />
-    <xacro:kinect_rgb_sensor_gazebo link_name="${name}_rgb" frame_name="${name}_rgb_optical_frame" camera_name="${name}_rgb" />
+    <xacro:kinect_ir_sensor_gazebo link_name="${camera_name}_ir" frame_name="${camera_name}_ir_optical_frame" camera_name="${camera_name}_ir" />
+    <xacro:kinect_rgb_sensor_gazebo link_name="${camera_name}_rgb" frame_name="${camera_name}_rgb_optical_frame" camera_name="${camera_name}_rgb" />
   </xacro:macro>
 </robot>

Commit message: [Fix] kinect coordination

File: robots/ubiquitous_display_for_gazebo.urdf.xacro (robot description, xacro)
@@ -9,5 +9,5 @@
   <xacro:hokuyo_utm30lx_model name="front_laser" parent="front_laser_adjuster_link" />
   <xacro:hokuyo_utm30lx_model name="rear_laser" parent="rear_laser_adjuster_link" />
-  <!--xacro:kinect2_for_gazebo_model name="ud_pt_" camera_name="camera"/-->
+  <xacro:kinect2_for_gazebo_model name="ud_pt_" camera_name="camera"/>
   <!-- =============== Gazebo =============== -->
   <gazebo>

File: urdf/sensor/kinect/kinect2_for_gazebo.urdf.xacro (robot description, xacro)
@@ -20,5 +20,5 @@
       <child link="${camera_name}_plate_link" />
     </joint>
-    <link name="${camera_name}_rgb_optical_frame">
+    <link name="${camera_name}_base_frame">
       <collision>
         <origin xyz="-1.56 0 0" rpy="0 0 0"/>
@@ -45,17 +45,24 @@
       </inertial>
     </link>
+    <link name="${camera_name}_rgb_optical_frame">
+    </link>
     <link name="${camera_name}_ir_optical_frame">
     </link>
-    <joint name="${camera_name}_plate_to_${camera_name}_rgb_optical_frame" type="fixed">
-      <origin xyz="0.095 0 0.08 " rpy="0 -1.57 -1.57" />
+    <joint name="${camera_name}_plate_to_${camera_name}_base_frame" type="fixed">
+      <origin xyz="0.095 0 0.035 " rpy="-1.56 0 0" />
       <parent link="${camera_name}_plate_link"/>
+      <child link="${camera_name}_base_frame"/>
+    </joint>
+    <joint name="${camera_name}_base_frame_to_${camera_name}_rgb_optical_frame" type="fixed">
+      <origin xyz="0 0 0.03 " rpy="-1.57 -1.57 -1.57" />
+      <parent link="${camera_name}_base_frame"/>
       <child link="${camera_name}_rgb_optical_frame"/>
     </joint>
     <joint name="${camera_name}_rgb_optical_frame_to_${camera_name}_ir_optical_frame" type="fixed">
-      <origin xyz="-0.0425 0 0.045 " rpy="-1.57 -1.57 -1.57" />
+      <origin xyz="0 0 -0.0425" rpy="0 0 0" />
       <parent link="${camera_name}_rgb_optical_frame"/>
       <child link="${camera_name}_ir_optical_frame"/>
     </joint>
-    <gazebo reference="${camera_name}_rgb_optical_frame">
+    <gazebo reference="${camera_name}_base_frame">
       <mu1>0.2</mu1>
       <mu2>0.2</mu2>

Commit message: [Fix] camera coordination for gazebo

File: robots/ubiquitous_display_for_gazebo.urdf.xacro (robot description, xacro)
@@ -6,8 +6,8 @@
   <xacro:include filename="$(find ubiquitous_display_description)/urdf/sensor/lrf/hokuyo_utm30lx.urdf.xacro"/>
   <xacro:include filename="$(find ubiquitous_display_description)/urdf/sensor/kinect/kinect2_for_gazebo.urdf.xacro"/>
-  <xacro:pantilt_model name="ud_pt_" parent="top_plate_link"/>
+  <xacro:pantilt_model name="pantilt" parent="top_plate_link"/>
   <xacro:hokuyo_utm30lx_model name="front_laser" parent="front_laser_adjuster_link" />
   <xacro:hokuyo_utm30lx_model name="rear_laser" parent="rear_laser_adjuster_link" />
-  <xacro:kinect2_for_gazebo_model name="ud_pt_" camera_name="camera"/>
+  <xacro:kinect2_for_gazebo_model camera_name="camera" parent="projector_link"/>
   <!-- =============== Gazebo =============== -->
   <gazebo>

File: urdf/sensor/kinect/kinect2_for_gazebo.urdf.xacro (robot description, xacro)
@@ -5,6 +5,6 @@
 <robot xmlns:xacro="http://www.ros.org/wiki/xacro" name="kinect2_for_gazebo">
   <xacro:include filename="$(find ubiquitous_display_description)/urdf/sensor/kinect/kinect2.gazebo.xacro"/>
-  <xacro:macro name="kinect2_for_gazebo_model" params="name camera_name">
-    <link name="${camera_name}_plate_link">
+  <xacro:macro name="kinect2_for_gazebo_model" params="camera_name parent">
+    <link name="kinect2_plate_link">
       <visual>
         <origin xyz="0 0 0" rpy="0 0 0" />
@@ -15,12 +15,12 @@
       </visual>
     </link>
-    <joint name="${name}projector_link_to_${camera_name}_plate_link" type="fixed">
-      <origin xyz="0.075 -0.11 0.135" rpy="0 0 3.14" />
-      <parent link="${name}projector_link" />
-      <child link="${camera_name}_plate_link" />
+    <joint name="${parent}_to_kinect2_plate_link" type="fixed">
+      <origin xyz="-0.075 0.11 0.135" rpy="0 0 0" />
+      <parent link="${parent}" />
+      <child link="kinect2_plate_link" />
     </joint>
     <link name="${camera_name}_base_frame">
       <collision>
-        <origin rpy="-1.56 0 0" xyz="0 0 0"/>
+        <origin rpy="0 0 0" xyz="0 0 0"/>
         <geometry>
           <box size="0.25 0.065 0.068"/>
@@ -28,5 +28,5 @@
       </collision>
       <visual>
-        <origin rpy="-1.56 0 0" xyz="0 0 0"/>
+        <origin rpy="0 0 0" xyz="0 0 0"/>
         <geometry>
             <!-- these meshes were exported in mm, so scale back to m -->
@@ -38,5 +38,5 @@
       <inertial>
         <mass value="0.2" />
-        <origin rpy="-1.56 0 0" xyz="0 0 0"/>
+        <origin rpy="0 0 0" xyz="0 0 0"/>
         <inertia
           ixx="0.00147" ixy="0" ixz="0"
@@ -49,16 +49,16 @@
     <link name="${camera_name}_ir_optical_frame">
     </link>
-    <joint name="${camera_name}_plate_to_${camera_name}_base_frame" type="fixed">
+    <joint name="kinect2_plate_link_to_${camera_name}_base_frame" type="fixed">
       <origin xyz="0.095 0 0.035 " rpy="-1.56 0 0" />
-      <parent link="${camera_name}_plate_link"/>
+      <parent link="kinect2_plate_link"/>
       <child link="${camera_name}_base_frame"/>
     </joint>
     <joint name="${camera_name}_base_frame_to_${camera_name}_rgb_optical_frame" type="fixed">
-      <origin xyz="0 0 0.03 " rpy="-1.57 -1.57 -1.57" />
+      <origin xyz="0 0 0.03 " rpy="0 -1.57 0" />
       <parent link="${camera_name}_base_frame"/>
       <child link="${camera_name}_rgb_optical_frame"/>
     </joint>
     <joint name="${camera_name}_rgb_optical_frame_to_${camera_name}_ir_optical_frame" type="fixed">
-      <origin xyz="0 0 -0.0425" rpy="0 0 0" />
+      <origin xyz="0 0 0.0425" rpy="0 0 0" />
       <parent link="${camera_name}_rgb_optical_frame"/>
       <child link="${camera_name}_ir_optical_frame"/>

Commit message: [Add] projector plugin

File: robots/ubiquitous_display_for_gazebo.urdf.xacro (robot description, xacro)
@@ -10,4 +10,6 @@
   <xacro:hokuyo_utm30lx_model name="rear_laser" parent="rear_laser_adjuster_link" />
   <xacro:kinect2_for_gazebo_model camera_name="camera" parent="projector_link"/>
+  <xacro:ubiquitous_display_transmission />
+  <xacro:pantilt_gazebo name="pantilt"/>
   <!-- =============== Gazebo =============== -->
   <gazebo>

File: urdf/pantilt/pantilt.gazebo.xacro (robot description, xacro)
@@ -22,5 +22,28 @@
     <material>Gazebo/LightGrey</material>
   </gazebo>
+  <gazebo reference="projector_gazebo_optical_frame">
+    <projector name="ud_projector">
+      <!-- setting the pose will produce glitches even when attached to a revolute joint -->
+      <pose>0 0 0 0 0 0</pose>
+      <texture>pop_gazebo.png</texture>
+      <!--texture>stereo_projection_pattern_high_res_red.png</texture-->
+      <fov>0.7</fov>
+      <near_clip>0.1</near_clip>
+      <far_clip>5.0</far_clip>
+    </projector>
+  </gazebo>
+  <gazebo>
+     <plugin filename="libgazebo_my_projector.so" name="projector">
+         <projector>projector_gazebo_optical_frame/ud_projector</projector>
+         <alwaysOn>true</alwaysOn>
+         <updateRate>10.0</updateRate>
+         <!-- Apparently the 2 lines below does not affect anything -->
+         <textureName>pop_gazebo.png</textureName>
+         <filterTextureName>pop_gazebo.png</filterTextureName>
+         <!-- end -->
+         <textureTopicName>texture</textureTopicName>
+         <projectorTopicName>image</projectorTopicName>
+     </plugin>
+  </gazebo>
 </xacro:macro>
-  <xacro:pantilt_gazebo name="pantilt"/>
 </robot>

File: urdf/pantilt/pantilt.transmission.xacro (robot description, xacro)
@@ -23,4 +23,3 @@
   </transmission>
 </xacro:macro>
-<xacro:ubiquitous_display_transmission />
 </robot>

File: urdf/pantilt/pantilt.urdf.xacro (robot description, xacro)
@@ -91,4 +91,5 @@
     </link>
     <link name="projector_optical_frame"/>
+    <link name="projector_gazebo_optical_frame"/>
     <joint name="${parent}_to_${name}base_link" type="fixed">
       <origin xyz="0 0 0.033 " rpy="0 0 0" />
@@ -125,4 +126,9 @@
       <child link="projector_optical_frame"/>
     </joint>
+    <joint name="projector_link_to_projector_gazebo_optical_frame" type="fixed">
+      <origin xyz="0 0 0 " rpy="1.57 0 0" />
+      <parent link="projector_link"/>
+      <child link="projector_gazebo_optical_frame"/>
+    </joint>
   </xacro:macro>
 </robot>
