Commit message: add interial and gazebo tag in pantilt files

File: robots/ubiquitous_display.urdf.xacro (robot description, xacro)
@@ -66,5 +66,5 @@
   <gazebo>
     <plugin name="gazebo_ros_control" filename="libgazebo_ros_control.so">
-      <robotNamespace>ubiquitous_display</robotNamespace>
+      <robotNamespace>/ubiquitous_display</robotNamespace>
       <robotSimType>gazebo_ros_control/DefaultRobotHWSim</robotSimType>
       <legacyModeNS>true</legacyModeNS>

File: urdf/pantilt/pantilt.gazebo.xacro (robot description, xacro)
@@ -1,14 +1,19 @@
 <?xml version="1.0"?>
-<xacro:macro name="ubiquitous_display_gazebo">
-<gazebo>
-  <plugin name="differential_drive_controller" filename="libgazebo_ros_diff_drive.so">
-    <leftJoint>left_wheel_joint</leftJoint>
-    <rightJoint>right_wheel_joint</rightJoint>
-    <robotBaseFrame>base_link</robotBaseFrame>
-    <wheelSeparation>0.108</wheelSeparation>
-    <wheelDiameter>0.024</wheelDiameter>
-    <publishWheelJointState>true</publishWheelJointState>
-    <legacyMode>false</legacyMode>
-  </plugin>
-</gazebo>
-</xacro>
+<robot name="pantilt_gazebo" xmlns:xacro="http://www.ros.org/wiki/xacro">
+<xacro:macro name="pantilt_gazebo" params="name">
+  <gazebo reference="${name}box_link">
+    <material>Gazebo/Grey</material>
+  </gazebo>
+  <gazebo reference="${name}plate_link">
+    <mu1>0.2</mu1>
+    <mu2>0.2</mu2>
+    <material>Gazebo/Grey</material>
+  </gazebo>
+  <gazebo reference="${name}projector_link">
+    <mu1>0.2</mu1>
+    <mu2>0.2</mu2>
+    <material>Gazebo/Grey</material>
+  </gazebo>
+</xacro:macro>
+  <xacro:pantilt_gazebo name="ud_pt_"/>
+</robot>

File: urdf/pantilt/pantilt.transmission.xacro (robot description, xacro)
@@ -1,3 +1,4 @@
 <?xml version="1.0"?>
+<robot name="pantilt_trans" xmlns:xacro="http://ros.org/wiki/xacro">
 <xacro:macro name="ubiquitous_display_transmission">
 <transmission name="pan_tran">
@@ -21,3 +22,4 @@
   </actuator>
 </transmission>
-</xacro>
+</xacro:macro>
+</robot>

File: urdf/pantilt/pantilt.urdf.xacro (robot description, xacro)
@@ -1,4 +1,6 @@
 <?xml version="1.0"?>
 <robot name="pantilt" xmlns:xacro="http://www.ros.org/wiki/xacro">
+  <xacro:include filename="$(find ubiquitous_display_description)/urdf/pantilt/pantilt.transmission.xacro"/>
+  <xacro:include filename="$(find ubiquitous_display_description)/urdf/pantilt/pantilt.gazebo.xacro"/>
   <xacro:property name="base_to_box_height" value="0.065"/>
   <xacro:property name="box_to_proj_height" value="0.17"/>
@@ -26,4 +28,12 @@
         <material name="gray"/>
       </visual>
+     <inertial>
+       <origin xyz="0 0 ${base_to_box_height/2}" rpy="0 0 0"/>
+       <mass value="1"/>
+       <inertia
+	    ixx="1.0" ixy="0.0" ixz="0.0"
+	    iyy="1.0" iyz="0.0"
+	    izz="1.0"/>
+     </inertial>
     </link>
     <link name="${name}plate_link">
@@ -35,4 +45,12 @@
         <material name="gray"/>
       </visual>
+     <inertial>
+       <origin xyz="0 0 0.0015" rpy="0 0 0"/>
+       <mass value="1"/>
+       <inertia
+	    ixx="1.0" ixy="0.0" ixz="0.0"
+	    iyy="1.0" iyz="0.0"
+	    izz="1.0"/>
+     </inertial>
     </link>
     <link name="left_pt_pillars" >
@@ -62,4 +80,12 @@
         <material name="gray"/>
       </visual>
+     <inertial>
+       <origin xyz="0 0 0.035" rpy="0 0 0"/>
+       <mass value="1"/>
+       <inertia
+	    ixx="1.0" ixy="0.0" ixz="0.0"
+	    iyy="1.0" iyz="0.0"
+	    izz="1.0"/>
+     </inertial>
     </link>
     <joint name="${name}base_joint" type="fixed">
@@ -75,4 +101,5 @@
       <axis xyz="0 0 1" />
       <limit lower="0" upper="2" effort="1" velocity="1"/>
+      <dynamics damping="0.7"/>
     </joint>
     <joint name="ud_pt_plate_link_to_left_pt_pillars" type="fixed">
@@ -92,4 +119,5 @@
       <axis xyz="1 0 0" />
       <limit lower="0" upper="2" effort="1" velocity="1"/>
+      <dynamics damping="0.7"/>
     </joint>
   </xacro:macro>

Commit message: [Fix] include <kinect2.xacro> file

File: robots/ubiquitous_display.urdf.xacro (robot description, xacro)
@@ -17,50 +17,7 @@
     <child link="ud_pt_base_link"/>
   </joint>
-  <link name="kinect2_plate_link">
-    <visual>
-      <origin xyz="0 0 0" rpy="0 0 0" />
-      <geometry>
-        <box size="0.25 0.015 0.01" />
-      </geometry>
-      <material name="gray"/>
-    </visual>
-  </link>
-  <joint name="ud_pt_projector_link_to_kinect2_plate_link" type="fixed">
-    <origin xyz="0.075 -0.11 0.135" rpy="0 0 3.14" />
-    <parent link="ud_pt_projector_link" />
-    <child link="kinect2_plate_link" />
-  </joint>
-  <link name="kinect2_rgb_optical_frame">
-    <visual>
-      <origin rpy="-1.56 0 0" xyz="0 0 0"/>
-      <geometry>
-          <!-- these meshes were exported in mm, so scale back to m -->
-        <mesh filename="package://ubiquitous_display_description/meshes/STL/kinect2_origin_on_rgb_optical_frame.stl" scale="0.001 0.001 0.001"/>
-        <!--box size="0.25 0.07 0.45" /-->
-      </geometry>
-      <material name="black"/>
-    </visual>
-  </link>
-  <link name="kinect2_ir_optical_frame">
-    <visual>
-      <origin rpy="0.075 0 0" xyz="0 0 0"/>
-      <geometry>
-        <sphere radius="0.0005"/>
-      </geometry>
-      <material name="black"/>
-    </visual>
-  </link>
-  <joint name="kinect2_plate_to_kinect2_rgb_optical_frame" type="fixed">
-    <origin xyz="0.095 0 0.035 " rpy="0 0 0" />
-    <parent link="kinect2_plate_link"/>
-    <child link="kinect2_rgb_optical_frame"/>
-  </joint>
-  <joint name="kinect2_rgb_optical_frame_to_kinect2_ir_optical_frame" type="fixed">
-    <origin xyz="-0.0425 0 0 " rpy="0 0 0" />
-    <parent link="kinect2_rgb_optical_frame"/>
-    <child link="kinect2_ir_optical_frame"/>
-  </joint>
   <xacro:hokuyo_utm30lx_model name="front_laser" parent="front_laser_adjuster_link" />
   <xacro:hokuyo_utm30lx_model name="rear_laser" parent="rear_laser_adjuster_link" />
+  <xacro:kinect2_model name="ud_pt_"/>
   <!-- =============== Gazebo =============== -->
   <gazebo>

File: urdf/sensor/kinect/kinect2.gazebo.xacro (robot description, xacro)
@@ -1,5 +1,5 @@
 <?xml version="1.0"?>
-<root xmlns:xacro="http://ros.org/wiki/xacro">
-	<xacro:macro name="kinect_ir_sensor" params="link_name frame_name camera_name">
+<robot xmlns:xacro="http://ros.org/wiki/xacro">
+	<xacro:macro name="kinect_ir_sensor_gazebo" params="link_name frame_name camera_name">
 		<gazebo reference="${link_name}">
 			<sensor type="depth" name="${link_name}_ir_sensor">
@@ -45,5 +45,5 @@
 		</gazebo>
 	</xacro:macro>
-	<xacro:macro name="kinect_rgb_sensor" params="link_name frame_name camera_name">
+	<xacro:macro name="kinect_rgb_sensor_gazebo" params="link_name frame_name camera_name">
 		<gazebo reference="${link_name}">
 			<sensor type="depth" name="${link_name}_rgb_sensor">
@@ -88,3 +88,3 @@
 		</gazebo>
 	</xacro:macro>
-</root>
+</robot>

File: urdf/sensor/kinect/kinect2.urdf.xacro (robot description, xacro)
@@ -4,23 +4,48 @@
 <!-- License: GPLv3+ -->
 <robot xmlns:xacro="http://www.ros.org/wiki/xacro" name="kinect2">
-  <xacro:macro name="kinect2_xacro" params="prefix parent *origin">
-    <material name="Kinect2Grey">
-      <color rgba="0.15 0.15 0.15 1.0"/>
-    </material>
-    <link name="${prefix}_kinect2_rgb_optical_frame">
+  <xacro:macro name="kinect2_model" params="name">
+    <link name="kinect2_plate_link">
       <visual>
-        <origin rpy="0 0 0" xyz="0 0 0"/>
+        <origin xyz="0 0 0" rpy="0 0 0" />
         <geometry>
-          <!-- these meshes were exported in mm, so scale back to m -->
-          <mesh filename="package://ubiquitous_display_description/meshes/STL/kinect2_origin_on_rgb_optical_frame.stl" scale="0.001 0.001 0.001"/>
+          <box size="0.25 0.015 0.01" />
         </geometry>
-        <material name="Kinect2Grey"/>
+        <material name="gray"/>
       </visual>
     </link>
-    <!-- Joint connecting the parent to our frame_in -->
-    <joint name="${prefix}_kinect2_in_joint" type="fixed">
-      <xacro:insert_block name="origin"/>
-      <parent link="${parent}"/>
-      <child link="${prefix}_kinect2_rgb_optical_frame"/>
+    <joint name="${name}projector_link_to_kinect2_plate_link" type="fixed">
+      <origin xyz="0.075 -0.11 0.135" rpy="0 0 3.14" />
+      <parent link="${name}projector_link" />
+      <child link="kinect2_plate_link" />
+    </joint>
+    <link name="kinect2_rgb_optical_frame">
+      <visual>
+        <origin rpy="-1.56 0 0" xyz="0 0 0"/>
+        <geometry>
+            <!-- these meshes were exported in mm, so scale back to m -->
+          <mesh filename="package://ubiquitous_display_description/meshes/STL/kinect2_origin_on_rgb_optical_frame.stl" scale="0.001 0.001 0.001"/>
+          <!--box size="0.25 0.07 0.45" /-->
+        </geometry>
+        <material name="black"/>
+      </visual>
+    </link>
+    <link name="kinect2_ir_optical_frame">
+      <visual>
+        <origin rpy="0.075 0 0" xyz="0 0 0"/>
+        <geometry>
+          <sphere radius="0.0005"/>
+        </geometry>
+        <material name="black"/>
+      </visual>
+    </link>
+    <joint name="kinect2_plate_to_kinect2_rgb_optical_frame" type="fixed">
+      <origin xyz="0.095 0 0.035 " rpy="0 0 0" />
+      <parent link="kinect2_plate_link"/>
+      <child link="kinect2_rgb_optical_frame"/>
+    </joint>
+    <joint name="kinect2_rgb_optical_frame_to_kinect2_ir_optical_frame" type="fixed">
+      <origin xyz="-0.0425 0 0 " rpy="0 0 0" />
+      <parent link="kinect2_rgb_optical_frame"/>
+      <child link="kinect2_ir_optical_frame"/>
     </joint>
   </xacro:macro>

Commit message: [Fix] pan and tilt joint setting

File: robots/ubiquitous_display.urdf.xacro (robot description, xacro)
@@ -13,5 +13,5 @@
   <!-- joint for body and pantilt-->
   <joint name="top_plate_link_to_ud_pt_base_link" type="fixed">
-    <origin xyz="0 0 0.0325 " rpy="0 0 0" />
+    <origin xyz="0 0 0.0325 " rpy="0 0 3.14" />
     <parent link="top_plate_link"/>
     <child link="ud_pt_base_link"/>

File: urdf/pantilt/pantilt.urdf.xacro (robot description, xacro)
@@ -39,5 +39,5 @@
     <link name="${name}plate_link">
       <visual>
-        <origin xyz="-0.075 0 0" rpy="0 0 0" />
+        <origin xyz="0.075 0 0" rpy="0 0 0" />
         <geometry>
           <box size="0.35 0.095 0.003" />
@@ -124,15 +124,15 @@
       <parent link="${name}plate_link"/>
       <child link="left_pt_pillars"/>
-      <origin xyz="0.09 0 0.1" rpy="0 0 0" />
+      <origin xyz="-0.09 0 0.1" rpy="0 0 0" />
     </joint>
     <joint name="${name}plate_link_to_right_pt_pillars" type="fixed">
       <parent link="${name}plate_link"/>
       <child link="right_pt_pillars"/>
-      <origin xyz="-0.24 0 0.1" rpy="0 0 0" />
+      <origin xyz="0.24 0 0.1" rpy="0 0 0" />
     </joint>
     <joint name="tilt_joint" type="revolute">
       <parent link="${name}plate_link"/>
       <child link="${name}projector_link"/>
-      <origin xyz="0 0 ${box_to_proj_height}" rpy="0 0 3.14" />
+      <origin xyz="0 0 ${box_to_proj_height}" rpy="0 0 0" />
       <axis xyz="1 0 0" />
       <limit lower="-0.2617" upper="1.3" effort="10" velocity="1"/>
@@ -143,5 +143,5 @@
       <parent link="${name}projector_link"/>
       <child link="${name}projector_optical_frame"/>
-      <origin xyz="0 -0.02 0" rpy="0 0 3.14" />
+      <origin xyz="0 -0.02 0" rpy="-1.56 0 3.14" />
     </joint>
   </xacro:macro>

Commit message: [Renmae] base_link and base_footprint from ud_

File: robots/ubiquitous_display.urdf.xacro (robot description, xacro)
@@ -6,15 +6,5 @@
   <xacro:include filename="$(find ubiquitous_display_description)/urdf/youbot/youbot_base_only.urdf.xacro"/>
   <xacro:include filename="$(find ubiquitous_display_description)/urdf/sensor/lrf/hokuyo_utm30lx.urdf.xacro"/>
-  <joint name="ud_base_link_to_bottom_pillars_link" type="fixed">
-    <origin xyz="0 0 0" rpy="0 0 0" />
-    <parent link="ud_base_link"/>
-    <child link="bottom_pillars_link"/>
-  </joint>
-  <!-- joint for body and pantilt-->
-  <joint name="top_plate_link_to_ud_pt_base_link" type="fixed">
-    <origin xyz="0 0 0.0325 " rpy="0 0 3.14" />
-    <parent link="top_plate_link"/>
-    <child link="ud_pt_base_link"/>
-  </joint>
+  <xacro:pantilt_name name="ud_pt_" parent="top_plate_link"/>
   <xacro:hokuyo_utm30lx_model name="front_laser" parent="front_laser_adjuster_link" />
   <xacro:hokuyo_utm30lx_model name="rear_laser" parent="rear_laser_adjuster_link" />

File: urdf/body/body.urdf.xacro (robot description, xacro)
@@ -77,4 +77,9 @@
   <!-- Bottom part -->
   <xacro:tower_template name="bottom" pillar_height="${bottom_pillar_height}"/>
+  <joint name="base_link_to_bottom_pillars_link" type="fixed">
+    <origin xyz="0 0 0" rpy="0 0 0" />
+    <parent link="base_link"/>
+    <child link="bottom_pillars_link"/>
+  </joint>
   <!-- Middle part -->
   <xacro:tower_template name="middle" pillar_height="${middle_pillar_height}"/>

File: urdf/pantilt/pantilt.urdf.xacro (robot description, xacro)
@@ -17,5 +17,5 @@
     <color rgba="0.7 0.7 0.7 1.0" />
   </material>
-  <xacro:macro name="pantilt_name" params="name">
+  <xacro:macro name="pantilt_name" params="name parent">
     <link name="${name}base_link" >
     </link>
@@ -106,4 +106,9 @@
     </link>
     <link name="${name}projector_optical_frame"/>
+    <joint name="top_plate_link_to_ud_pt_base_link" type="fixed">
+      <origin xyz="0 0 0.0325 " rpy="0 0 3.14" />
+      <parent link="${parent}"/>
+      <child link="${name}base_link"/>
+    </joint>
     <joint name="${name}base_joint" type="fixed">
       <parent link="${name}base_link"/>
@@ -146,4 +151,3 @@
     </joint>
   </xacro:macro>
-  <xacro:pantilt_name name="ud_pt_"/>
 </robot>

File: urdf/youbot/youbot_base_only.urdf.xacro (robot description, xacro)
@@ -18,4 +18,4 @@
        the origin block defines where the component is w.r.t its parent (in this case the parent
        is the world frame). For more, see http://www.ros.org/wiki/xacro -->
-  <xacro:youbot_base name="ud_base"/>
+  <xacro:youbot_base name="base"/>
 </robot>

Commit message: [Fix] remove gzebo.xacro file in kinect2.urdf.xacro

File: robots/ubiquitous_display.urdf.xacro (robot description, xacro)
@@ -10,5 +10,5 @@
   <xacro:hokuyo_utm30lx_model name="rear_laser" parent="rear_laser_adjuster_link" />
   <xacro:kinect2_model name="ud_pt_" parent="kinect2_plate_link"/>
-  <xacro:kinect2_for_gazebo name="" rgb_parent="kinect2_rgb_optical_frame" depth_parent="kinect2_ir_optical_frame"/>
+  <!--xacro:kinect2_for_gazebo_model name="" rgb_parent="kinect2_rgb_optical_frame" depth_parent="kinect2_ir_optical_frame"/-->
   <!-- =============== Gazebo =============== -->
   <gazebo>

File: urdf/sensor/kinect/kinect2.urdf.xacro (robot description, xacro)
@@ -4,5 +4,4 @@
 <!-- License: GPLv3+ -->
 <robot xmlns:xacro="http://www.ros.org/wiki/xacro" name="kinect2">
-  <xacro:include filename="$(find ubiquitous_display_description)/urdf/sensor/kinect/kinect2.gazebo.xacro"/>
   <xacro:macro name="kinect2_model" params="name parent">
     <link name="kinect2_plate_link">
@@ -64,7 +63,4 @@
       <child link="kinect2_ir_optical_frame"/>
     </joint>
-    <!--<xacro:camera_gazebo link_name="kinect2_rgb" frame_name="kinect2_rgb_optical_frame"/>-->
-    <xacro:kinect_ir_sensor_gazebo link_name="kinect2_ir" frame_name="kinect2_ir_optical_frame" camera_name="kinect2" />
-    <xacro:kinect_rgb_sensor_gazebo link_name="kinect2_rgb" frame_name="kinect2_rgb_optical_frame" camera_name="kinect2" />
   </xacro:macro>
 </robot>

File: urdf/sensor/kinect/kinect2_for_gazebo.urdf.xacro (robot description, xacro)
@@ -5,44 +5,5 @@
 <robot xmlns:xacro="http://www.ros.org/wiki/xacro" name="kinect2">
   <xacro:include filename="$(find ubiquitous_display_description)/urdf/sensor/kinect/kinect2.gazebo.xacro"/>
-  <xacro:macro name="kinect2_model" params="name parent">
-    <link name="kinect2_plate_link">
-      <visual>
-        <origin xyz="0 0 0" rpy="0 0 0" />
-        <geometry>
-          <box size="0.25 0.015 0.01" />
-        </geometry>
-        <material name="gray"/>
-      </visual>
-    </link>
-    <joint name="${name}projector_link_to_kinect2_plate_link" type="fixed">
-      <origin xyz="0.075 -0.11 0.135" rpy="0 0 3.14" />
-      <parent link="${name}projector_link" />
-      <child link="${parent}" />
-    </joint>
-    <link name="kinect2_rgb_optical_frame">
-      <collision>
-        <origin xyz="-1.56 0 0" rpy="0 0 0"/>
-        <geometry>
-          <box size="0.25 0.065 0.068"/>
-        </geometry>
-      </collision>
-      <visual>
-        <origin rpy="-1.56 0 0" xyz="0 0 0"/>
-        <geometry>
-            <!-- these meshes were exported in mm, so scale back to m -->
-          <mesh filename="package://ubiquitous_display_description/meshes/STL/kinect2_origin_on_rgb_optical_frame.stl" scale="0.001 0.001 0.001"/>
-          <!--box size="0.25 0.07 0.6" /-->
-        </geometry>
-        <material name="black"/>
-      </visual>
-      <inertial>
-        <mass value="0.2" />
-        <origin xyz="-1.56 0 0" rpy="0 0 0"/>
-        <inertia
-          ixx="0.00147" ixy="0" ixz="0"
-          iyy="0.01112" iyz="0"
-          izz="0.01118" />
-      </inertial>
-    </link>
+  <xacro:macro name="kinect2_for_gazebo_model" params="name rgb_parent depth_parent">
     <link name="kinect2_ir_optical_frame">
       <visual>

Commit message: [Fix] camera_rgb_optical_link and camera_ir_optical_link

File: robots/ubiquitous_display.urdf.xacro (robot description, xacro)
@@ -6,9 +6,10 @@
   <xacro:include filename="$(find ubiquitous_display_description)/urdf/youbot/youbot_base_only.urdf.xacro"/>
   <xacro:include filename="$(find ubiquitous_display_description)/urdf/sensor/lrf/hokuyo_utm30lx.urdf.xacro"/>
+  <xacro:include filename="$(find ubiquitous_display_description)/urdf/sensor/kinect/kinect2_for_gazebo.urdf.xacro"/>
   <xacro:pantilt_model name="ud_pt_" parent="top_plate_link"/>
   <xacro:hokuyo_utm30lx_model name="front_laser" parent="front_laser_adjuster_link" />
   <xacro:hokuyo_utm30lx_model name="rear_laser" parent="rear_laser_adjuster_link" />
   <xacro:kinect2_model name="ud_pt_" parent="kinect2_plate_link"/>
-  <!--xacro:kinect2_for_gazebo_model name="" rgb_parent="kinect2_rgb_optical_frame" depth_parent="kinect2_ir_optical_frame"/-->
+  <xacro:kinect2_for_gazebo_model name="camera" rgb_parent="kinect2_rgb_optical_frame" depth_parent="kinect2_ir_optical_frame"/>
   <!-- =============== Gazebo =============== -->
   <gazebo>

File: urdf/sensor/kinect/kinect2_for_gazebo.urdf.xacro (robot description, xacro)
@@ -3,8 +3,8 @@
 <!-- Copyright Universitaet Bremen - Instititute for Artificial Intelligence. Author: Alexis Maldonado -->
 <!-- License: GPLv3+ -->
-<robot xmlns:xacro="http://www.ros.org/wiki/xacro" name="kinect2">
+<robot xmlns:xacro="http://www.ros.org/wiki/xacro" name="kinect2_for_gazebo">
   <xacro:include filename="$(find ubiquitous_display_description)/urdf/sensor/kinect/kinect2.gazebo.xacro"/>
   <xacro:macro name="kinect2_for_gazebo_model" params="name rgb_parent depth_parent">
-    <link name="kinect2_ir_optical_frame">
+    <link name="${name}_rgb_optical_frame">
       <visual>
         <origin rpy="0 0 0" xyz="0 0 0"/>
@@ -15,17 +15,26 @@
       </visual>
     </link>
-    <joint name="kinect2_plate_to_kinect2_rgb_optical_frame" type="fixed">
-      <origin xyz="0.095 0 0.035 " rpy="-1.56 0 0" />
-      <parent link="kinect2_plate_link"/>
-      <child link="kinect2_rgb_optical_frame"/>
+    <link name="${name}_ir_optical_frame">
+      <visual>
+        <origin rpy="0 0 0" xyz="0 0 0"/>
+        <geometry>
+          <sphere radius="0.0005"/>
+        </geometry>
+        <material name="black"/>
+      </visual>
+    </link>
+    <joint name="kinect2_rgb_optical_frame_to_${name}_rgb_optical_frame" type="fixed">
+      <origin xyz="0 0 0 " rpy="1.56 0 0" />
+      <parent link="${rgb_parent}"/>
+      <child link="${name}_rgb_optical_frame"/>
     </joint>
-    <joint name="kinect2_rgb_optical_frame_to_kinect2_ir_optical_frame" type="fixed">
-      <origin xyz="-0.0425 0 0 " rpy="0 0 0" />
-      <parent link="kinect2_rgb_optical_frame"/>
-      <child link="kinect2_ir_optical_frame"/>
+    <joint name="kinect2_ir_optical_frame_to_${name}_ir_optical_frame" type="fixed">
+      <origin xyz="0 0 0 " rpy="1.56 0 0" />
+      <parent link="${depth_parent}"/>
+      <child link="${name}_ir_optical_frame"/>
     </joint>
     <!--<xacro:camera_gazebo link_name="kinect2_rgb" frame_name="kinect2_rgb_optical_frame"/>-->
-    <xacro:kinect_ir_sensor_gazebo link_name="kinect2_ir" frame_name="kinect2_ir_optical_frame" camera_name="kinect2" />
-    <xacro:kinect_rgb_sensor_gazebo link_name="kinect2_rgb" frame_name="kinect2_rgb_optical_frame" camera_name="kinect2" />
+    <xacro:kinect_ir_sensor_gazebo link_name="${name}_ir" frame_name="${name}_ir_optical_frame" camera_name="${name}" />
+    <xacro:kinect_rgb_sensor_gazebo link_name="${name}_rgb" frame_name="${name}_rgb_optical_frame" camera_name="${name}" />
   </xacro:macro>
 </robot>
