Commit message: [Fix] Delete old link

File: robots/ubiquitous_display.urdf.xacro (robot description, xacro)
@@ -6,8 +6,8 @@
   <xacro:include filename="$(find ubiquitous_display_description)/urdf/youbot/youbot_base_only.urdf.xacro"/>
   <xacro:include filename="$(find ubiquitous_display_description)/urdf/sensor/lrf/hokuyo_utm30lx.urdf.xacro"/>
-  <xacro:pantilt_model name="ud_pt_" parent="top_plate_link"/>
+  <xacro:pantilt_model name="pantilt" parent="top_plate_link"/>
   <xacro:hokuyo_utm30lx_model name="front_laser" parent="front_laser_adjuster_link" />
   <xacro:hokuyo_utm30lx_model name="rear_laser" parent="rear_laser_adjuster_link" />
-  <xacro:kinect2_model name="ud_pt_" parent="kinect2_plate_link"/>
+  <xacro:kinect2_model parent="projector_link"/>
   <!-- =============== Gazebo =============== -->
   <gazebo>

File: urdf/pantilt/pantilt.gazebo.xacro (robot description, xacro)
@@ -2,8 +2,20 @@
 <robot name="pantilt_gazebo" xmlns:xacro="http://www.ros.org/wiki/xacro">
 <xacro:macro name="pantilt_gazebo" params="name">
-  <gazebo reference="${name}box_link">
+  <gazebo reference="${name}base_link">
+    <mu1>0.2</mu1>
+    <mu2>0.2</mu2>
     <material>Gazebo/LightGrey</material>
   </gazebo>
-  <gazebo reference="${name}plate_link">
+  <gazebo reference="tilt_link">
+    <mu1>0.2</mu1>
+    <mu2>0.2</mu2>
+    <material>Gazebo/LightGrey</material>
+  </gazebo>
+  <gazebo reference="pan_link">
+    <mu1>0.2</mu1>
+    <mu2>0.2</mu2>
+    <material>Gazebo/LightGrey</material>
+  </gazebo>
+  <gazebo reference="projector_link">
     <mu1>0.2</mu1>
     <mu2>0.2</mu2>
@@ -11,4 +23,4 @@
   </gazebo>
 </xacro:macro>
-  <xacro:pantilt_gazebo name="ud_pt_"/>
+  <xacro:pantilt_gazebo name="pantilt"/>
 </robot>

File: urdf/pantilt/pantilt.urdf.xacro (robot description, xacro)
@@ -19,6 +19,4 @@
   <xacro:macro name="pantilt_model" params="name parent">
     <link name="${name}base_link" >
-    </link>
-    <link name="${name}box_link" >
       <visual>
         <origin xyz="0 0 0" rpy="0 0 0" />
@@ -38,5 +36,5 @@
      </inertial>
     </link>
-    <link name="${name}plate_link">
+    <link name="pan_link">
       <visual>
         <origin xyz="0 0 0" rpy="0 0 0" />
@@ -56,49 +54,15 @@
      </inertial>
     </link>
-    <!--link name="left_pt_pillars" >
-      <visual>
-        <origin xyz="0 0 0" rpy="0 0 0" />
-        <geometry>
-          <box size="0.01 0.05 0.20" />
-        </geometry>
-        <material name="gray" />
-      </visual>
-     <inertial>
-       <origin xyz="0 0 0.01" rpy="0 0 0"/>
-       <mass value="0.06"/>
-       <inertia
-	    ixx="0.00708" ixy="0.0" ixz="0.0"
-	    iyy="0.00043" iyz="0.0"
-	    izz="0.00668"/>
-     </inertial>
-    </link>
-    <link name="right_pt_pillars" >
-      <visual>
-        <origin xyz="0 0 0" rpy="0 0 0" />
-        <geometry>
-          <box size="0.01 0.05 0.20" />
-        </geometry>
-        <material name="gray" />
-      </visual>
-     <inertial>
-       <origin xyz="0 0 0.01" rpy="0 0 0"/>
-       <mass value="0.06"/>
-       <inertia
-	    ixx="1.0" ixy="0.0" ixz="0.0"
-	    iyy="1.0" iyz="0.0"
-	    izz="1.0"/>
-     </inertial>
-   </link-->
-    <link name="${name}projector_link">
+    <link name="tilt_link">
       <visual>
         <origin xyz="0 0 0" rpy="0 0 0" />
         <geometry>
           <!--box size="0.24 0.17 0.07" /-->
-          <mesh filename="package://ubiquitous_display_description/meshes/STL/ud_pt_tilt_with_projector.stl" scale="0.001 0.001 0.001"/>
+          <mesh filename="package://ubiquitous_display_description/meshes/STL/ud_pt_tilt.stl" scale="0.001 0.001 0.001"/>
         </geometry>
         <material name="gray"/>
       </visual>
      <inertial>
-       <origin xyz="0 0 0.035" rpy="0 0 0"/>
+       <origin xyz="0 0 0" rpy="0 0 0"/>
        <mass value="2"/>
        <inertia
@@ -108,19 +72,32 @@
      </inertial>
     </link>
-    <link name="${name}projector_optical_frame"/>
-    <joint name="top_plate_link_to_ud_pt_base_link" type="fixed">
-      <origin xyz="0 0 0.0325 " rpy="0 0 0" />
+    <link name="projector_link">
+      <visual>
+        <origin xyz="0 0 0" rpy="0 0 0" />
+        <geometry>
+          <!--box size="0.24 0.17 0.07" /-->
+          <mesh filename="package://ubiquitous_display_description/meshes/STL/projector.stl" scale="0.001 0.001 0.001"/>
+        </geometry>
+        <material name="gray"/>
+      </visual>
+     <inertial>
+       <origin xyz="0 0 0" rpy="0 0 0"/>
+       <mass value="2"/>
+       <inertia
+      ixx="0.00536" ixy="0.0" ixz="0.0"
+      iyy="0.01441" iyz="0.0"
+      izz="0.01041"/>
+     </inertial>
+    </link>
+    <link name="projector_optical_frame"/>
+    <joint name="${parent}_to_${name}base_link" type="fixed">
+      <origin xyz="0 0 0.033 " rpy="0 0 0" />
       <parent link="${parent}"/>
       <child link="${name}base_link"/>
     </joint>
-    <joint name="${name}base_joint" type="fixed">
-      <parent link="${name}base_link"/>
-      <child link="${name}box_link"/>
-      <origin xyz="0 0 0" rpy="0 0 0" />
-    </joint>
     <!--name of pan_joint and tilt_joint depend pantilt.yaml-->
     <joint name="pan_joint" type="revolute">
-      <parent link="${name}box_link"/>
-      <child link="${name}plate_link"/>
+      <parent link="${name}base_link"/>
+      <child link="pan_link"/>
       <origin xyz="0 0 ${base_to_box_height/2}" rpy="0 0 0" />
       <axis xyz="0 0 1" />
@@ -129,27 +106,22 @@
       <dynamics damping="0.7"/>
     </joint>
-    <!--joint name="${name}plate_link_to_left_pt_pillars" type="fixed">
-      <parent link="${name}plate_link"/>
-      <child link="left_pt_pillars"/>
-      <origin xyz="-0.09 0 0.1" rpy="0 0 0" />
-    </joint>
-    <joint name="${name}plate_link_to_right_pt_pillars" type="fixed">
-      <parent link="${name}plate_link"/>
-      <child link="right_pt_pillars"/>
-      <origin xyz="0.24 0 0.1" rpy="0 0 0" />
-    </joint-->
     <joint name="tilt_joint" type="revolute">
-      <parent link="${name}plate_link"/>
-      <child link="${name}projector_link"/>
-      <origin xyz="0 0 ${box_to_proj_height}" rpy="0 0 3.14" />
-      <axis xyz="1 0 0" />
+      <parent link="pan_link"/>
+      <child link="tilt_link"/>
+      <origin xyz="0.0905 0 0.170" rpy="0 -1.57 0" />
+      <axis xyz="0 0 1" />
       <limit lower="-0.2617" upper="1.3" effort="10" velocity="1"/>
       <!--<safety_controller k_velocity="10" k_position="15" soft_lower_limit="-2.0" soft_upper_limit="0.5" />-->
       <dynamics damping="0.7"/>
     </joint>
-    <joint name="${name}projector_link_to_${name}projector_optical_frame" type="fixed">
-      <parent link="${name}projector_link"/>
-      <child link="${name}projector_optical_frame"/>
-      <origin xyz="0 -0.02 0" rpy="-1.56 0 3.14" />
+    <joint name="tilt_link_to_projector_link" type="fixed">
+      <origin xyz="0 0 0.093 " rpy="0 1.57 0" />
+      <parent link="tilt_link"/>
+      <child link="projector_link"/>
+    </joint>
+    <joint name="projector_link_to_projector_optical_frame" type="fixed">
+      <origin xyz="0 0.0805 0 " rpy="-1.57 0 0" />
+      <parent link="projector_link"/>
+      <child link="projector_optical_frame"/>
     </joint>
   </xacro:macro>

File: urdf/sensor/kinect/kinect2.urdf.xacro (robot description, xacro)
@@ -4,5 +4,5 @@
 <!-- License: GPLv3+ -->
 <robot xmlns:xacro="http://www.ros.org/wiki/xacro" name="kinect2">
-  <xacro:macro name="kinect2_model" params="name parent">
+  <xacro:macro name="kinect2_model" params="parent">
     <link name="kinect2_plate_link">
       <visual>
@@ -14,8 +14,8 @@
       </visual>
     </link>
-    <joint name="${name}projector_link_to_kinect2_plate_link" type="fixed">
-      <origin xyz="0.075 -0.11 0.135" rpy="0 0 3.14" />
-      <parent link="${name}projector_link" />
-      <child link="${parent}" />
+    <joint name="${parent}_to_kinect2_plate_link" type="fixed">
+      <origin xyz="-0.075 0.11 0.135" rpy="0 0 0" />
+      <parent link="${parent}" />
+      <child link="kinect2_plate_link" />
     </joint>
     <link name="kinect2_rgb_optical_frame">

Commit message: [Edit] select visual argument (hokuyo-utm30lx)

File: robots/ubiquitous_display.urdf.xacro (robot description, xacro)
@@ -7,6 +7,6 @@
   <xacro:include filename="$(find ubiquitous_display_description)/urdf/sensor/lrf/hokuyo_utm30lx.urdf.xacro"/>
   <xacro:pantilt_model name="pantilt_" parent="top_plate_link"/>
-  <xacro:hokuyo_utm30lx_model name="front_laser" parent="front_laser_adjuster_link" />
-  <xacro:hokuyo_utm30lx_model name="rear_laser" parent="rear_laser_adjuster_link" />
+  <xacro:hokuyo_utm30lx_model name="front_laser" parent="front_laser_adjuster_link" visual="false"/>
+  <xacro:hokuyo_utm30lx_model name="rear_laser" parent="rear_laser_adjuster_link" visual="false"/>
   <xacro:kinect2_model parent="projector_link"/>
   <!-- =============== Gazebo =============== -->

File: robots/ubiquitous_display_for_gazebo.urdf.xacro (robot description, xacro)
@@ -7,6 +7,6 @@
   <xacro:include filename="$(find ubiquitous_display_description)/urdf/sensor/kinect/kinect2_for_gazebo.urdf.xacro"/>
   <xacro:pantilt_model name="pantilt_" parent="top_plate_link"/>
-  <xacro:hokuyo_utm30lx_model name="front_laser" parent="front_laser_adjuster_link" />
-  <xacro:hokuyo_utm30lx_model name="rear_laser" parent="rear_laser_adjuster_link" />
+  <xacro:hokuyo_utm30lx_model name="front_laser" parent="front_laser_adjuster_link" visual="true"/>
+  <xacro:hokuyo_utm30lx_model name="rear_laser" parent="rear_laser_adjuster_link" visual="false"/>
   <xacro:kinect2_for_gazebo_model camera_name="camera" parent="projector_link"/>
   <xacro:ubiquitous_display_transmission />

File: urdf/sensor/lrf/hokuyo_utm30lx.gazebo.xacro (robot description, xacro)
@@ -35,10 +35,10 @@
     </gazebo>
   </xacro:macro>
-  <xacro:macro name="hokuyo_utm30lx_gpu" params="name ray_count min_angle max_angle">
+  <xacro:macro name="hokuyo_utm30lx_gpu" params="name ray_count min_angle max_angle visual">
     <gazebo reference="${name}_frame">
       <sensor type="gpu_ray" name="${name}">
         <update_rate>40</update_rate>
         <pose>0 0 0 0 0 0</pose>
-        <visualize>false</visualize>
+        <visualize>${visual}</visualize>
         <ray>
           <scan>

File: urdf/sensor/lrf/hokuyo_utm30lx.urdf.xacro (robot description, xacro)
@@ -3,5 +3,5 @@
     <xacro:include filename="$(find ubiquitous_display_description)/urdf/sensor/lrf/hokuyo_utm30lx.gazebo.xacro"/>
     <xacro:property name="M_PI" value="3.1415926535897931" />
-    <xacro:macro name="hokuyo_utm30lx_model" params="name parent">
+    <xacro:macro name="hokuyo_utm30lx_model" params="name parent visual">
       <joint name="${name}_joint" type="fixed">
         <!--xacro:insert_block name="origin" /-->
@@ -30,5 +30,5 @@
         </collision>
       </link>
-      <xacro:hokuyo_utm30lx_gpu name="${name}" ray_count="1080" min_angle="-135" max_angle="135" />
+      <xacro:hokuyo_utm30lx_gpu name="${name}" ray_count="1080" min_angle="-135" max_angle="135" visual="${visual}"/>
     </xacro:macro>
 </robot>
