Commit message: [Add] gazebo plaugin (camera_rgb_optical_frame)

File: urdf/sensor/kinect/kinect2_for_gazebo.urdf.xacro (robot description, xacro)
@@ -57,4 +57,9 @@
       <child link="${camera_name}_ir_optical_frame"/>
     </joint>
+    <gazebo reference="${camera_name}_rgb_optical_frame">
+      <mu1>0.2</mu1>
+      <mu2>0.2</mu2>
+      <material>Gazebo/Black</material>
+    </gazebo>
     <!--<xacro:camera_gazebo link_name="kinect2_rgb" frame_name="kinect2_rgb_optical_frame"/>-->
     <xacro:kinect_ir_sensor_gazebo link_name="${camera_name}_ir" frame_name="${camera_name}_ir_optical_frame" camera_name="${camera_name}_ir" />
