Commit message: [Add] kinect frame's collision and inertial

File: urdf/sensor/kinect/kinect2.urdf.xacro (robot description, xacro)
@@ -21,4 +21,10 @@
     </joint>
     <link name="kinect2_rgb_optical_frame">
+      <collision>
+        <origin xyz="0 0 0" rpy="0 0 0"/>
+        <geometry>
+          <box size="0.25 0.065 0.068"/>
+        </geometry>
+      </collision>
       <visual>
         <origin rpy="-1.56 0 0" xyz="0 0 0"/>
@@ -26,8 +32,16 @@
             <!-- these meshes were exported in mm, so scale back to m -->
           <mesh filename="package://ubiquitous_display_description/meshes/STL/kinect2_origin_on_rgb_optical_frame.stl" scale="0.001 0.001 0.001"/>
-          <!--box size="0.25 0.07 0.45" /-->
+          <!--box size="0.25 0.07 0.6" /-->
         </geometry>
         <material name="black"/>
       </visual>
+      <inertial>
+        <mass value="0.2" />
+        <origin xyz="0 0 0" rpy="0 0 0"/>
+        <inertia
+          ixx="0.00147" ixy="0" ixz="0"
+          iyy="0.01112" iyz="0"
+          izz="0.01118" />
+      </inertial>
     </link>
     <link name="kinect2_ir_optical_frame">
@@ -50,6 +64,6 @@
       <child link="kinect2_ir_optical_frame"/>
     </joint>
-    <xacro:kinect_ir_sensor_gazebo link_name="kinect2_ir_optical_frame" frame_name="kinect2_ir_optical_frame" camera_name="ubiquitous_display" />
-    <xacro:kinect_rgb_sensor_gazebo link_name="kinect2_rgb_optical_frame" frame_name="kinect2_rgb_optical_frame" camera_name="ubiquitous_display" />
+    <!--<xacro:kinect_ir_sensor_gazebo link_name="kinect2_ir_optical_frame" frame_name="kinect2_ir_optical_frame" camera_name="ir" />-->
+    <xacro:kinect_rgb_sensor_gazebo link_name="kinect2_rgb_optical_frame" frame_name="kinect2_rgb_optical_frame" camera_name="rgb" />
   </xacro:macro>
 </robot>

Commit message: [Fix] kinect2 optical frame cordination

File: urdf/sensor/kinect/kinect2.urdf.xacro (robot description, xacro)
@@ -55,5 +55,5 @@
     </link>
     <joint name="kinect2_plate_to_kinect2_rgb_optical_frame" type="fixed">
-      <origin xyz="0.095 0 0.035 " rpy="0 0 0" />
+      <origin xyz="0.095 0 0.035 " rpy="-1.56 0 0" />
       <parent link="kinect2_plate_link"/>
       <child link="kinect2_rgb_optical_frame"/>

Commit message: [Delete] ir_optical <visual> tag

File: urdf/sensor/kinect/kinect2.urdf.xacro (robot description, xacro)
@@ -45,11 +45,4 @@
     </link>
     <link name="kinect2_ir_optical_frame">
-      <visual>
-        <origin rpy="0 0 0" xyz="0 0 0"/>
-        <geometry>
-          <sphere radius="0.0005"/>
-        </geometry>
-        <material name="black"/>
-      </visual>
     </link>
     <joint name="kinect2_plate_to_kinect2_rgb_optical_frame" type="fixed">

Commit message: [Fix] origin value (rpy, xyz)

File: urdf/sensor/kinect/kinect2.urdf.xacro (robot description, xacro)
@@ -21,5 +21,5 @@
     <link name="kinect2_rgb_optical_frame">
       <collision>
-        <origin xyz="-1.56 0 0" rpy="0 0 0"/>
+        <origin rpy="-1.56 0 0" xyz="0 0 0"/>
         <geometry>
           <box size="0.25 0.065 0.068"/>
@@ -37,5 +37,5 @@
       <inertial>
         <mass value="0.2" />
-        <origin xyz="-1.56 0 0" rpy="0 0 0"/>
+        <origin rpy="-1.56 0 0" xyz="0 0 0"/>
         <inertia
           ixx="0.00147" ixy="0" ixz="0"

File: urdf/sensor/kinect/kinect2_for_gazebo.urdf.xacro (robot description, xacro)
@@ -22,5 +22,5 @@
     <link name="${camera_name}_base_frame">
       <collision>
-        <origin xyz="-1.56 0 0" rpy="0 0 0"/>
+        <origin rpy="-1.56 0 0" xyz="0 0 0"/>
         <geometry>
           <box size="0.25 0.065 0.068"/>
@@ -38,5 +38,5 @@
       <inertial>
         <mass value="0.2" />
-        <origin xyz="-1.56 0 0" rpy="0 0 0"/>
+        <origin rpy="-1.56 0 0" xyz="0 0 0"/>
         <inertia
           ixx="0.00147" ixy="0" ixz="0"
