Commit message: [Add]kinect.gazebo.xacro

File: urdf/sensor/kinect/kinect2.gazebo.xacro (robot description, xacro)
@@ -0,0 +1,90 @@
+<?xml version="1.0"?>
+<root xmlns:xacro="http://ros.org/wiki/xacro">
+	<xacro:macro name="kinect_ir_sensor" params="link_name frame_name camera_name">
+		<gazebo reference="${link_name}">
+			<sensor type="depth" name="${link_name}_ir_sensor">
+				<always_on>true</always_on>
+				<update_rate>1.0</update_rate>
+				<camera>
+					<horizontal_fov>${57.0*PI/180.0}</horizontal_fov>
+						<image>
+							<format>L8</format>
+							<width>640</width>
+							<height>480</height>
+						</image>
+					<clip>
+						<near>1.2</near>
+						<far>3.5</far>
+					</clip>
+				</camera>
+				<plugin name="${link_name}_controller" filename="libgazebo_ros_openni_kinect.so">
+					<baseline>0.2</baseline>
+					<alwaysOn>true</alwaysOn>
+					<updateRate>1.0</updateRate>
+					<cameraName>${camera_name}_ir</cameraName>
+					<imageTopicName>/${camera_name}/depth/image_raw</imageTopicName>
+					<cameraInfoTopicName>/${camera_name}/depth/camera_info</cameraInfoTopicName>
+					<depthImageTopicName>/${camera_name}/depth/image_raw</depthImageTopicName>
+					<depthImageCameraInfoTopicName>/${camera_name}/depth/camera_info</depthImageCameraInfoTopicName>
+					<pointCloudTopicName>/${camera_name}/depth/points</pointCloudTopicName>
+					<frameName>${frame_name}</frameName>
+					<pointCloudCutoff>0.5</pointCloudCutoff>
+					<distortionK1>0.00000001</distortionK1>
+					<distortionK2>0.00000001</distortionK2>
+					<distortionK3>0.00000001</distortionK3>
+					<distortionT1>0.00000001</distortionT1>
+					<distortionT2>0.00000001</distortionT2>
+					<CxPrime>0</CxPrime>
+					<Cx>0</Cx>
+					<Cy>0</Cy>
+					<focalLength>0</focalLength>
+					<hackBaseline>0</hackBaseline>
+				</plugin>
+			</sensor>
+			<material value="Gazebo/Red"/>
+		</gazebo>
+	</xacro:macro>
+	<xacro:macro name="kinect_rgb_sensor" params="link_name frame_name camera_name">
+		<gazebo reference="${link_name}">
+			<sensor type="depth" name="${link_name}_rgb_sensor">
+				<always_on>true</always_on>
+				<update_rate>1.0</update_rate>
+				<camera>
+					<horizontal_fov>${57.0*PI/180.0}</horizontal_fov>
+					<image>
+						<format>R8G8B8</format>
+						<width>640</width>
+						<height>480</height>
+					</image>
+					<clip>
+						<near>1.2</near>
+						<far>3.5</far>
+					</clip>
+				</camera>
+				<plugin name="${link_name}_controller" filename="libgazebo_ros_openni_kinect.so">
+					<alwaysOn>true</alwaysOn>
+					<updateRate>1.0</updateRate>
+					<cameraName>${camera_name}_rgb</cameraName>
+					<imageTopicName>/${camera_name}/rgb/image_raw</imageTopicName>
+					<cameraInfoTopicName>/${camera_name}/rgb/camera_info</cameraInfoTopicName>
+					<depthImageTopicName>/${camera_name}/depth/image_raw</depthImageTopicName>
+					<depthImageCameraInfoTopicName>/${camera_name}/depth/camera_info</depthImageCameraInfoTopicName>
+					<pointCloudTopicName>/${camera_name}/depth_registered/points</pointCloudTopicName>
+					<frameName>${frame_name}</frameName>
+					<pointCloudCutoff>0.5</pointCloudCutoff>
+					<distortionK1>0.00000001</distortionK1>
+					<distortionK2>0.00000001</distortionK2>
+					<distortionK3>0.00000001</distortionK3>
+					<distortionT1>0.00000001</distortionT1>
+					<distortionT2>0.00000001</distortionT2>
+					<CxPrime>0</CxPrime>
+					<Cx>0</Cx>
+					<Cy>0</Cy>
+					<focalLength>0</focalLength>
+					<hackBaseline>0</hackBaseline>
+				</plugin>
+			</sensor>
+			<material value="Gazebo/Red"/>
+		</gazebo>
+	</xacro:macro>
+</root>

Commit message: [Add] kinect <gazebo> tag

File: urdf/sensor/kinect/kinect2.gazebo.xacro (robot description, xacro)
@@ -1,48 +1,48 @@
 <?xml version="1.0"?>
-<robot xmlns:xacro="http://ros.org/wiki/xacro">
-	<xacro:macro name="kinect_ir_sensor_gazebo" params="link_name frame_name camera_name">
-		<gazebo reference="${link_name}">
-			<sensor type="depth" name="${link_name}_ir_sensor">
-				<always_on>true</always_on>
-				<update_rate>1.0</update_rate>
-				<camera>
-					<horizontal_fov>${57.0*PI/180.0}</horizontal_fov>
-						<image>
-							<format>L8</format>
-							<width>640</width>
-							<height>480</height>
-						</image>
-					<clip>
-						<near>1.2</near>
-						<far>3.5</far>
-					</clip>
-				</camera>
-				<plugin name="${link_name}_controller" filename="libgazebo_ros_openni_kinect.so">
-					<baseline>0.2</baseline>
-					<alwaysOn>true</alwaysOn>
-					<updateRate>1.0</updateRate>
-					<cameraName>${camera_name}_ir</cameraName>
-					<imageTopicName>/${camera_name}/depth/image_raw</imageTopicName>
-					<cameraInfoTopicName>/${camera_name}/depth/camera_info</cameraInfoTopicName>
-					<depthImageTopicName>/${camera_name}/depth/image_raw</depthImageTopicName>
-					<depthImageCameraInfoTopicName>/${camera_name}/depth/camera_info</depthImageCameraInfoTopicName>
-					<pointCloudTopicName>/${camera_name}/depth/points</pointCloudTopicName>
-					<frameName>${frame_name}</frameName>
-					<pointCloudCutoff>0.5</pointCloudCutoff>
-					<distortionK1>0.00000001</distortionK1>
-					<distortionK2>0.00000001</distortionK2>
-					<distortionK3>0.00000001</distortionK3>
-					<distortionT1>0.00000001</distortionT1>
-					<distortionT2>0.00000001</distortionT2>
-					<CxPrime>0</CxPrime>
-					<Cx>0</Cx>
-					<Cy>0</Cy>
-					<focalLength>0</focalLength>
-					<hackBaseline>0</hackBaseline>
-				</plugin>
-			</sensor>
-			<material value="Gazebo/Red"/>
-		</gazebo>
-	</xacro:macro>
+<robot xmlns:xacro="http://www.ros.org/wiki/xacro" name="kinect2_gazebo">
+  <xacro:macro name="kinect_ir_sensor_gazebo" params="link_name frame_name camera_name">
+    <gazebo reference="${link_name}">
+      <sensor type="depth" name="${link_name}_ir_sensor">
+        <always_on>true</always_on>
+        <update_rate>1.0</update_rate>
+        <camera>
+          <horizontal_fov>${57.0*M_PI/180.0}</horizontal_fov>
+            <image>
+              <format>L8</format>
+              <width>640</width>
+              <height>480</height>
+            </image>
+          <clip>
+            <near>1.2</near>
+            <far>3.5</far>
+          </clip>
+        </camera>
+        <plugin name="${link_name}_controller" filename="libgazebo_ros_openni_kinect.so">
+          <baseline>0.2</baseline>
+          <alwaysOn>true</alwaysOn>
+          <updateRate>1.0</updateRate>
+          <cameraName>${camera_name}_ir</cameraName>
+          <imageTopicName>/${camera_name}/depth/image_raw</imageTopicName>
+          <cameraInfoTopicName>/${camera_name}/depth/camera_info</cameraInfoTopicName>
+          <depthImageTopicName>/${camera_name}/depth/image_raw</depthImageTopicName>
+          <depthImageCameraInfoTopicName>/${camera_name}/depth/camera_info</depthImageCameraInfoTopicName>
+          <pointCloudTopicName>/${camera_name}/depth/points</pointCloudTopicName>
+          <frameName>${frame_name}</frameName>
+          <pointCloudCutoff>0.5</pointCloudCutoff>
+          <distortionK1>0.00000001</distortionK1>
+          <distortionK2>0.00000001</distortionK2>
+          <distortionK3>0.00000001</distortionK3>
+          <distortionT1>0.00000001</distortionT1>
+          <distortionT2>0.00000001</distortionT2>
+          <CxPrime>0</CxPrime>
+          <Cx>0</Cx>
+          <Cy>0</Cy>
+          <focalLength>0</focalLength>
+          <hackBaseline>0</hackBaseline>
+        </plugin>
+      </sensor>
+      <material value="Gazebo/Red"/>
+    </gazebo>
+  </xacro:macro>
 	<xacro:macro name="kinect_rgb_sensor_gazebo" params="link_name frame_name camera_name">
 		<gazebo reference="${link_name}">
@@ -51,5 +51,5 @@
 				<update_rate>1.0</update_rate>
 				<camera>
-					<horizontal_fov>${57.0*PI/180.0}</horizontal_fov>
+					<horizontal_fov>${57.0*M_PI/180.0}</horizontal_fov>
 					<image>
 						<format>R8G8B8</format>

File: urdf/sensor/kinect/kinect2.urdf.xacro (robot description, xacro)
@@ -4,4 +4,5 @@
 <!-- License: GPLv3+ -->
 <robot xmlns:xacro="http://www.ros.org/wiki/xacro" name="kinect2">
+  <xacro:include filename="$(find ubiquitous_display_description)/urdf/sensor/kinect/kinect2.gazebo.xacro"/>
   <xacro:macro name="kinect2_model" params="name">
     <link name="kinect2_plate_link">
@@ -49,4 +50,6 @@
       <child link="kinect2_ir_optical_frame"/>
     </joint>
+    <xacro:kinect_ir_sensor_gazebo link_name="kinect2_ir_optical_frame" frame_name="none" camera_name="none" />
+    <xacro:kinect_rgb_sensor_gazebo link_name="kinect2_rgb_optical_frame" frame_name="none" camera_name="none" />
   </xacro:macro>
 </robot>

Commit message: [Change] kinect frame color

File: urdf/sensor/kinect/kinect2.gazebo.xacro (robot description, xacro)
@@ -42,5 +42,5 @@
         </plugin>
       </sensor>
-      <material value="Gazebo/Red"/>
+      <material value="Gazebo/Black"/>
     </gazebo>
   </xacro:macro>
@@ -85,5 +85,5 @@
 				</plugin>
 			</sensor>
-			<material value="Gazebo/Red"/>
+			<material value="Gazebo/Black"/>
 		</gazebo>
 	</xacro:macro>

File: urdf/sensor/kinect/kinect2.urdf.xacro (robot description, xacro)
@@ -50,6 +50,6 @@
       <child link="kinect2_ir_optical_frame"/>
     </joint>
-    <xacro:kinect_ir_sensor_gazebo link_name="kinect2_ir_optical_frame" frame_name="none" camera_name="none" />
-    <xacro:kinect_rgb_sensor_gazebo link_name="kinect2_rgb_optical_frame" frame_name="none" camera_name="none" />
+    <xacro:kinect_ir_sensor_gazebo link_name="kinect2_ir_optical_frame" frame_name="kinect2_ir_optical_frame" camera_name="ubiquitous_display" />
+    <xacro:kinect_rgb_sensor_gazebo link_name="kinect2_rgb_optical_frame" frame_name="kinect2_rgb_optical_frame" camera_name="ubiquitous_display" />
   </xacro:macro>
 </robot>

Commit message: [Add] libgazebo_ros_camera.so

File: urdf/sensor/kinect/kinect2.gazebo.xacro (robot description, xacro)
@@ -2,5 +2,5 @@
 <robot xmlns:xacro="http://www.ros.org/wiki/xacro" name="kinect2_gazebo">
   <xacro:macro name="kinect_ir_sensor_gazebo" params="link_name frame_name camera_name">
-    <gazebo reference="${link_name}">
+    <gazebo reference="${link_name}_optical_frame">
       <sensor type="depth" name="${link_name}_ir_sensor">
         <always_on>true</always_on>
@@ -46,6 +46,6 @@
   </xacro:macro>
 	<xacro:macro name="kinect_rgb_sensor_gazebo" params="link_name frame_name camera_name">
-		<gazebo reference="${link_name}">
-			<sensor type="depth" name="${link_name}_rgb_sensor">
+		<gazebo reference="${link_name}_optical_frame">
+			<sensor type="depth" name="${link_name}_sensor">
 				<always_on>true</always_on>
 				<update_rate>1.0</update_rate>
@@ -88,3 +88,45 @@
 		</gazebo>
 	</xacro:macro>
+  <xacro:macro name="camera_gazebo" params="link_name frame_name">
+      <gazebo reference="${link_name}_optical_frame">
+      <sensor type="camera" name="camera1">
+        <update_rate>30.0</update_rate>
+        <camera name="head">
+          <horizontal_fov>1.3962634</horizontal_fov>
+          <image>
+            <width>800</width>
+            <height>800</height>
+            <format>R8G8B8</format>
+          </image>
+          <clip>
+            <near>0.02</near>
+            <far>300</far>
+          </clip>
+          <noise>
+            <type>gaussian</type>
+            <!-- Noise is sampled independently per pixel on each frame.
+                 That pixel's noise value is added to each of its color
+                 channels, which at that point lie in the range [0,1]. -->
+            <mean>0.0</mean>
+            <stddev>0.007</stddev>
+          </noise>
+        </camera>
+        <plugin name="camera_controller" filename="libgazebo_ros_camera.so">
+          <alwaysOn>true</alwaysOn>
+          <updateRate>0.0</updateRate>
+          <cameraName>rrbot/camera1</cameraName>
+          <imageTopicName>image_raw</imageTopicName>
+          <cameraInfoTopicName>camera_info</cameraInfoTopicName>
+          <frameName>${frame_name}</frameName>
+          <hackBaseline>0.07</hackBaseline>
+          <distortionK1>0.0</distortionK1>
+          <distortionK2>0.0</distortionK2>
+          <distortionK3>0.0</distortionK3>
+          <distortionT1>0.0</distortionT1>
+          <distortionT2>0.0</distortionT2>
+        </plugin>
+      </sensor>
+      <material value="Gazebo/Black"/>
+    </gazebo>
+  </xacro:macro>
 </robot>

File: urdf/sensor/kinect/kinect2.urdf.xacro (robot description, xacro)
@@ -64,6 +64,7 @@
       <child link="kinect2_ir_optical_frame"/>
     </joint>
+    <xacro:camera_gazebo link_name="kinect2_rgb" frame_name="kinect2_rgb_optical_frame"/>
     <!--<xacro:kinect_ir_sensor_gazebo link_name="kinect2_ir_optical_frame" frame_name="kinect2_ir_optical_frame" camera_name="ir" />-->
-    <xacro:kinect_rgb_sensor_gazebo link_name="kinect2_rgb_optical_frame" frame_name="kinect2_rgb_optical_frame" camera_name="rgb" />
+    <!--<xacro:kinect_rgb_sensor_gazebo link_name="kinect2_rgb_optical_frame" frame_name="kinect2_rgb_optical_frame" camera_name="rgb" />-->
   </xacro:macro>
 </robot>

Commit message: [Delete] camera_gazebo

File: urdf/sensor/kinect/kinect2.gazebo.xacro (robot description, xacro)
@@ -90,45 +90,3 @@
 		</gazebo>
 	</xacro:macro>
-  <xacro:macro name="camera_gazebo" params="link_name frame_name">
-      <gazebo reference="${link_name}_optical_frame">
-      <sensor type="camera" name="camera1">
-        <update_rate>30.0</update_rate>
-        <camera name="head">
-          <horizontal_fov>1.3962634</horizontal_fov>
-          <image>
-            <width>800</width>
-            <height>800</height>
-            <format>R8G8B8</format>
-          </image>
-          <clip>
-            <near>0.02</near>
-            <far>300</far>
-          </clip>
-          <noise>
-            <type>gaussian</type>
-            <!-- Noise is sampled independently per pixel on each frame.
-                 That pixel's noise value is added to each of its color
-                 channels, which at that point lie in the range [0,1]. -->
-            <mean>0.0</mean>
-            <stddev>0.007</stddev>
-          </noise>
-        </camera>
-        <plugin name="camera_controller" filename="libgazebo_ros_camera.so">
-          <alwaysOn>true</alwaysOn>
-          <updateRate>0.0</updateRate>
-          <cameraName>rrbot/camera1</cameraName>
-          <imageTopicName>image_raw</imageTopicName>
-          <cameraInfoTopicName>camera_info</cameraInfoTopicName>
-          <frameName>${frame_name}</frameName>
-          <hackBaseline>0.07</hackBaseline>
-          <distortionK1>0.0</distortionK1>
-          <distortionK2>0.0</distortionK2>
-          <distortionK3>0.0</distortionK3>
-          <distortionT1>0.0</distortionT1>
-          <distortionT2>0.0</distortionT2>
-        </plugin>
-      </sensor>
-      <material value="Gazebo/Black"/>
-    </gazebo>
-  </xacro:macro>
 </robot>

Commit message: [Fix] kinect plugin and kinect2 frame name

File: urdf/sensor/kinect/kinect2.gazebo.xacro (robot description, xacro)
@@ -2,5 +2,5 @@
 <robot xmlns:xacro="http://www.ros.org/wiki/xacro" name="kinect2_gazebo">
   <xacro:macro name="kinect_ir_sensor_gazebo" params="link_name frame_name camera_name">
-    <gazebo reference="${link_name}_optical_frame">
+    <gazebo reference="${link_name}_link">
       <sensor type="depth" name="${link_name}_sensor">
         <always_on>true</always_on>
@@ -46,5 +46,5 @@
   </xacro:macro>
 	<xacro:macro name="kinect_rgb_sensor_gazebo" params="link_name frame_name camera_name">
-		<gazebo reference="${link_name}_optical_frame">
+		<gazebo reference="${link_name}_link">
 			<sensor type="depth" name="${link_name}_sensor">
 				<always_on>true</always_on>

File: urdf/sensor/kinect/kinect2_for_gazebo.urdf.xacro (robot description, xacro)
@@ -45,8 +45,10 @@
       </inertial>
     </link>
-    <link name="${camera_name}_rgb_optical_frame">
+    <link name="${camera_name}_rgb_link">
     </link>
-    <link name="${camera_name}_ir_optical_frame">
+    <link name="${camera_name}_ir_link">
     </link>
+    <link name="kinect2_rgb_optical_frame"/>
+    <link name="kinect2_ir_optical_frame"/>
     <joint name="kinect2_plate_link_to_${camera_name}_base_frame" type="fixed">
       <origin xyz="0.095 0 0.035 " rpy="-1.56 0 0" />
@@ -54,13 +56,23 @@
       <child link="${camera_name}_base_frame"/>
     </joint>
-    <joint name="${camera_name}_base_frame_to_${camera_name}_rgb_optical_frame" type="fixed">
+    <joint name="${camera_name}_base_frame_to_${camera_name}_rgb_link" type="fixed">
       <origin xyz="0 0 0.03 " rpy="0 -1.57 0" />
       <parent link="${camera_name}_base_frame"/>
-      <child link="${camera_name}_rgb_optical_frame"/>
+      <child link="${camera_name}_rgb_link"/>
     </joint>
-    <joint name="${camera_name}_rgb_optical_frame_to_${camera_name}_ir_optical_frame" type="fixed">
+    <joint name="${camera_name}_rgb_link_to_${camera_name}_ir_link" type="fixed">
       <origin xyz="0 0 0.0425" rpy="0 0 0" />
-      <parent link="${camera_name}_rgb_optical_frame"/>
-      <child link="${camera_name}_ir_optical_frame"/>
+      <parent link="${camera_name}_rgb_link"/>
+      <child link="${camera_name}_ir_link"/>
+    </joint>
+    <joint name="${camera_name}_rgb_link_to_kinect2_rgb_optical_frame" type="fixed">
+      <origin rpy="${M_PI/2} ${M_PI} ${M_PI/2}"/>
+      <parent link="${camera_name}_rgb_link"/>
+      <child link="kinect2_rgb_optical_frame"/>
+    </joint>
+    <joint name="${camera_name}_ir_link_to_kinect2_ir_optical_frame" type="fixed">
+      <origin rpy="${M_PI/2} ${M_PI} ${M_PI/2}"/>
+      <parent link="${camera_name}_ir_link"/>
+      <child link="kinect2_ir_optical_frame"/>
     </joint>
     <gazebo reference="${camera_name}_base_frame">
@@ -70,6 +82,6 @@
     </gazebo>
     <!--<xacro:camera_gazebo link_name="kinect2_rgb" frame_name="kinect2_rgb_optical_frame"/>-->
-    <xacro:kinect_ir_sensor_gazebo link_name="${camera_name}_ir" frame_name="${camera_name}_ir_optical_frame" camera_name="${camera_name}_ir" />
-    <xacro:kinect_rgb_sensor_gazebo link_name="${camera_name}_rgb" frame_name="${camera_name}_rgb_optical_frame" camera_name="${camera_name}_rgb" />
+    <xacro:kinect_ir_sensor_gazebo link_name="${camera_name}_ir" frame_name="kinect2_ir_optical_frame" camera_name="${camera_name}_ir" />
+    <xacro:kinect_rgb_sensor_gazebo link_name="${camera_name}_rgb" frame_name="kinect2_rgb_optical_frame" camera_name="${camera_name}_rgb" />
   </xacro:macro>
 </robot>
