Commit message: [Complete] all stl file

File: urdf/body/body.gazebo.xacro (robot description, xacro)
@@ -5,5 +5,5 @@
     <mu1>0.2</mu1>
     <mu2>0.2</mu2>
-    <material>Gazebo/Grey</material>
+    <material>Gazebo/LightGrey</material>
   </gazebo>
 </xacro:macro>

File: urdf/body/body.urdf.xacro (robot description, xacro)
@@ -41,5 +41,5 @@
         <geometry>
           <!--box size="${plate_len_x} ${plate_len_y} ${plate_len_z}"/-->
-          <mesh filename="package://ubiquitous_display_description/meshes/STL/base_plate.stl" scale="0.001 0.001 0.001"/>
+          <mesh filename="package://ubiquitous_display_description/meshes/STL/${name}_plate.stl" scale="0.001 0.001 0.001"/>
         </geometry>
         <origin xyz="0 0 -${plate_len_z/2}"/>

File: urdf/materials.urdf.xacro (robot description, xacro)
@@ -26,5 +26,5 @@
   </material>
   <material name="LightGrey">
-    <color rgba="0.82 0.82 0.82 1.0"/>
+    <color rgba="0.80 0.80 0.80 1.0"/>
   </material>
 </robot>

File: urdf/pantilt/pantilt.gazebo.xacro (robot description, xacro)
@@ -3,25 +3,10 @@
 <xacro:macro name="pantilt_gazebo" params="name">
   <gazebo reference="${name}box_link">
-    <material>Gazebo/Grey</material>
+    <material>Gazebo/LightGrey</material>
   </gazebo>
   <gazebo reference="${name}plate_link">
     <mu1>0.2</mu1>
     <mu2>0.2</mu2>
-    <material>Gazebo/Grey</material>
-  </gazebo>
-  <gazebo reference="${name}projector_link">
-    <mu1>0.2</mu1>
-    <mu2>0.2</mu2>
-    <material>Gazebo/Grey</material>
-  </gazebo>
-  <gazebo reference="left_pt_pillars">
-    <mu1>0.2</mu1>
-    <mu2>0.2</mu2>
-    <material>Gazebo/Grey</material>
-  </gazebo>
-  <gazebo reference="right_pt_pillars">
-    <mu1>0.2</mu1>
-    <mu2>0.2</mu2>
-    <material>Gazebo/Grey</material>
+    <material>Gazebo/LightGrey</material>
   </gazebo>
 </xacro:macro>

File: urdf/pantilt/pantilt.urdf.xacro (robot description, xacro)
@@ -110,5 +110,5 @@
     <link name="${name}projector_optical_frame"/>
     <joint name="top_plate_link_to_ud_pt_base_link" type="fixed">
-      <origin xyz="0 0 0.0325 " rpy="0 0 3.14" />
+      <origin xyz="0 0 0.0325 " rpy="0 0 0" />
       <parent link="${parent}"/>
       <child link="${name}base_link"/>
@@ -142,5 +142,5 @@
       <parent link="${name}plate_link"/>
       <child link="${name}projector_link"/>
-      <origin xyz="0 0 ${box_to_proj_height}" rpy="0 0 0" />
+      <origin xyz="0 0 ${box_to_proj_height}" rpy="0 0 3.14" />
       <axis xyz="1 0 0" />
       <limit lower="-0.2617" upper="1.3" effort="10" velocity="1"/>

Commit message: [Edit] include DAE files

File: urdf/body/body.gazebo.xacro (robot description, xacro)
@@ -5,5 +5,5 @@
     <mu1>0.2</mu1>
     <mu2>0.2</mu2>
-    <material>Gazebo/LightGrey</material>
+    <!--material>Gazebo/LightGrey</material-->
   </gazebo>
 </xacro:macro>

File: urdf/body/body.urdf.xacro (robot description, xacro)
@@ -41,5 +41,5 @@
         <geometry>
           <!--box size="${plate_len_x} ${plate_len_y} ${plate_len_z}"/-->
-          <mesh filename="package://ubiquitous_display_description/meshes/STL/${name}_plate.stl" scale="0.001 0.001 0.001"/>
+          <mesh filename="package://ubiquitous_display_description/meshes/DAE/${name}_plate.dae" scale="0.001 0.001 0.001"/>
         </geometry>
         <origin xyz="0 0 -${plate_len_z/2}"/>
