Commit message: [Delete] ros_controller tag in youbot_base_only.urdf.xacro

File: urdf/body/body.urdf.xacro (robot description, xacro)
@@ -66,11 +66,4 @@
           <box size="${bar_len_x} ${bar_len_y} ${bar_len_z}"/>
         </geometry>
-        <origin xyz="${-bar_len_x/2} ${adjuster_width/2} ${bar_len_z/2}"/>
-        <material name="white" />
-      </visual>
-      <visual>
-        <geometry>
-          <box size="${bar_len_x} ${bar_len_y} ${bar_len_z}"/>
-        </geometry>
         <origin xyz="${-bar_len_x/2} ${-adjuster_width/2} ${bar_len_z/2}"/>
         <material name="white" />

File: urdf/youbot/youbot_base_only.urdf.xacro (robot description, xacro)
@@ -9,5 +9,5 @@
   <xacro:include filename="$(find ubiquitous_display_description)/urdf/materials.urdf.xacro" />
   <!-- controller manager -->
-  <xacro:include filename="$(find ubiquitous_display_description)/urdf/youbot/ros_controller.urdf.xacro" />
+  <!--<xacro:include filename="$(find ubiquitous_display_description)/urdf/youbot/ros_controller.urdf.xacro" />-->
   <!-- Now we can start using the macros xacro:included above to define the actual youbot -->
   <!-- The first use of a macro.  This one was defined in base.urdf.xacro above.

Commit message: [Fix] height joint

File: urdf/body/body.urdf.xacro (robot description, xacro)
@@ -3,5 +3,5 @@
   <xacro:include filename="$(find ubiquitous_display_description)/urdf/body/body.gazebo.xacro"/>
   <!-- Definition of various sizes -->
-  <xacro:property name="bottom_pillar_height" value="0.1"/>
+  <xacro:property name="bottom_pillar_height" value="0.14"/>
   <xacro:property name="middle_pillar_height" value="0.157"/>
   <xacro:property name="top_pillar_height" value="0.435"/>

File: urdf/sensor/kinect/kinect2.urdf.xacro (robot description, xacro)
@@ -22,5 +22,5 @@
     <link name="kinect2_rgb_optical_frame">
       <collision>
-        <origin xyz="0 0 0" rpy="0 0 0"/>
+        <origin xyz="-1.56 0 0" rpy="0 0 0"/>
         <geometry>
           <box size="0.25 0.065 0.068"/>
@@ -28,5 +28,5 @@
       </collision>
       <visual>
-        <origin rpy="0 0 0" xyz="0 0 0"/>
+        <origin rpy="-1.56 0 0" xyz="0 0 0"/>
         <geometry>
             <!-- these meshes were exported in mm, so scale back to m -->
@@ -38,5 +38,5 @@
       <inertial>
         <mass value="0.2" />
-        <origin xyz="0 0 0" rpy="0 0 0"/>
+        <origin xyz="-1.56 0 0" rpy="0 0 0"/>
         <inertia
           ixx="0.00147" ixy="0" ixz="0"

File: urdf/youbot/base.urdf.xacro (robot description, xacro)
@@ -51,5 +51,5 @@
     </link>
     <joint name="${name}_footprint_joint" type="fixed">
-      <origin xyz="0 0 0" rpy="0 0 0"/>
+      <origin xyz="0 0 0.08" rpy="0 0 0"/>
       <child link="${name}_link"/>
       <parent link="${name}_footprint"/>

Commit message: [Add] base_scan frame for lrf merge

File: urdf/body/body.urdf.xacro (robot description, xacro)
@@ -74,4 +74,33 @@
     </link>
   </xacro:macro>
+  <xacro:macro name="base_scan_model" params="name parent">
+    <joint name="${name}_scan_joint" type="fixed">
+      <!--xacro:insert_block name="origin" /-->
+      <origin xyz="-0.029 0 0.067" rpy="0 0 0"/>
+      <parent link="${parent}"/>
+      <child link="${name}_scan"/>
+    </joint>
+    <link name="${name}_scan">
+      <inertial>
+        <mass value="0.270" />
+        <origin xyz="0 0 0" rpy="0 0 0" />
+        <inertia ixx="2.632e-4" ixy="0" ixz="0" iyy="2.632e-4" iyz="0" izz="1.62e-4" />
+      </inertial>
+      <visual>
+        <origin xyz="0 0 0" rpy="0 0 0" />
+        <geometry>
+        <!--mesh filename="package://ubiquitous_display_description/meshes/DAE/hokuyo_utm_30lx.dae"/-->
+      </geometry>
+      </visual>
+      <collision>
+        <origin xyz="0 0 -0.0115" rpy="0 0 0" />
+        <geometry>
+        <box size="0.058 0.058 0.087" />
+        <!--<mesh filename="package://hector_sensors_description/meshes/hokuyo_utm30lx/hokuyo_utm_30lx.stl"/>-->
+      </geometry>
+      </collision>
+    </link>
+    <xacro:hokuyo_utm30lx_gazebo name="${name}" ray_count="1080" min_angle="-135" max_angle="135" />
+  </xacro:macro>
   <!-- Body -->
   <!-- Bottom part -->
@@ -111,3 +140,11 @@
   <child link="rear_laser_adjuster_link"/>
   </joint>
+  <!-- SCAN_FRAME for lrf_merger -->
+  <xacro:laser_adjuster_template name="base"/>
+  <joint name="base_scan_adjuster_joint" type="fixed">
+    <origin xyz="0 0 0" rpy="0 0 0"/>
+    <parent link="bottom_plate_link"/>
+    <child link="base_laser_adjuster_link"/>
+  </joint>
+  <xacro:base_scan_model name="base" parent="base_laser_adjuster_link"/>
 </robot>

Commit message: [Add] gazebo tag of base_scan

File: urdf/body/body.urdf.xacro (robot description, xacro)
@@ -77,5 +77,5 @@
     <joint name="${name}_scan_joint" type="fixed">
       <!--xacro:insert_block name="origin" /-->
-      <origin xyz="-0.029 0 0.067" rpy="0 0 0"/>
+      <origin xyz="0 0 0.067" rpy="0 0 0"/>
       <parent link="${parent}"/>
       <child link="${name}_scan"/>
@@ -90,6 +90,7 @@
         <origin xyz="0 0 0" rpy="0 0 0" />
         <geometry>
-        <!--mesh filename="package://ubiquitous_display_description/meshes/DAE/hokuyo_utm_30lx.dae"/-->
-      </geometry>
+          <sphere radius="0.01"/>
+        </geometry>
+        <material name="green"/>
       </visual>
       <collision>
@@ -100,4 +101,9 @@
       </geometry>
       </collision>
+      <gazebo reference="${name}_scan">
+        <mu1>0.2</mu1>
+        <mu2>0.2</mu2>
+        <material>Gazebo/Green</material>
+      </gazebo>
     </link>
     <xacro:hokuyo_utm30lx_gazebo name="${name}" ray_count="1080" min_angle="-135" max_angle="135" />
@@ -142,4 +148,5 @@
   <!-- SCAN_FRAME for lrf_merger -->
   <xacro:laser_adjuster_template name="base"/>
+  <xacro:laser_adjuster_template_gazebo name="base"/>
   <joint name="base_scan_adjuster_joint" type="fixed">
     <origin xyz="0 0 0" rpy="0 0 0"/>

Commit message: [Fix] laser_adjuster_template macro

File: urdf/body/body.urdf.xacro (robot description, xacro)
@@ -65,4 +65,11 @@
   <xacro:macro name="laser_adjuster_template" params="name">
     <link name="${name}_laser_adjuster_link">
+      <visual>
+        <geometry>
+          <box size="${bar_len_x} ${bar_len_y} ${bar_len_z}"/>
+        </geometry>
+        <origin xyz="${-bar_len_x/2} ${adjuster_width/2} ${bar_len_z/2}"/>
+        <material name="white" />
+      </visual>
       <visual>
         <geometry>

Commit message: [Remove] <visual> tag

File: urdf/body/body.urdf.xacro (robot description, xacro)
@@ -82,4 +82,20 @@
   </xacro:macro>
   <xacro:macro name="base_scan_model" params="name parent">
+    <link name="${name}_laser_adjuster_link">
+      <!--visual>
+        <geometry>
+          <box size="${bar_len_x} ${bar_len_y} ${bar_len_z}"/>
+        </geometry>
+        <origin xyz="${-bar_len_x/2} ${adjuster_width/2} ${bar_len_z/2}"/>
+        <material name="white" />
+      </visual-->
+      <!--visual>
+        <geometry>
+          <box size="${bar_len_x} ${bar_len_y} ${bar_len_z}"/>
+        </geometry>
+        <origin xyz="${-bar_len_x/2} ${-adjuster_width/2} ${bar_len_z/2}"/>
+        <material name="white" />
+      </visual-->
+    </link>
     <joint name="${name}_scan_joint" type="fixed">
       <!--xacro:insert_block name="origin" /-->
@@ -94,5 +110,5 @@
         <inertia ixx="2.632e-4" ixy="0" ixz="0" iyy="2.632e-4" iyz="0" izz="1.62e-4" />
       </inertial>
-      <visual>
+      <!--visual>
         <origin xyz="0 0 0" rpy="0 0 0" />
         <geometry>
@@ -100,5 +116,5 @@
         </geometry>
         <material name="green"/>
-      </visual>
+      </visual-->
       <collision>
         <origin xyz="0 0 -0.0115" rpy="0 0 0" />
@@ -153,6 +169,4 @@
   </joint>
   <!-- SCAN_FRAME for lrf_merger -->
-  <xacro:laser_adjuster_template name="base"/>
-  <xacro:laser_adjuster_template_gazebo name="base"/>
   <joint name="base_scan_adjuster_joint" type="fixed">
     <origin xyz="0 0 0" rpy="0 0 0"/>

Commit message: [Add] all stl file in xacro file

File: urdf/body/body.urdf.xacro (robot description, xacro)
@@ -6,5 +6,5 @@
   <xacro:property name="middle_pillar_height" value="0.157"/>
   <xacro:property name="top_pillar_height" value="0.435"/>
-  <xacro:property name="pillar_radius" value="0.01"/>
+  <xacro:property name="pillar_radius" value="0.008"/>
   <xacro:property name="pillar_offset_x" value="0.21"/>
   <xacro:property name="pillar_offset_y" value="0.06"/>
@@ -40,5 +40,6 @@
       <visual>
         <geometry>
-          <box size="${plate_len_x} ${plate_len_y} ${plate_len_z}"/>
+          <!--box size="${plate_len_x} ${plate_len_y} ${plate_len_z}"/-->
+          <mesh filename="package://ubiquitous_display_description/meshes/STL/base_plate.stl" scale="0.001 0.001 0.001"/>
         </geometry>
         <origin xyz="0 0 -${plate_len_z/2}"/>

File: urdf/pantilt/pantilt.urdf.xacro (robot description, xacro)
@@ -3,5 +3,5 @@
   <xacro:include filename="$(find ubiquitous_display_description)/urdf/pantilt/pantilt.transmission.xacro"/>
   <xacro:include filename="$(find ubiquitous_display_description)/urdf/pantilt/pantilt.gazebo.xacro"/>
-  <xacro:property name="base_to_box_height" value="0.065"/>
+  <xacro:property name="base_to_box_height" value="0.066"/>
   <xacro:property name="box_to_proj_height" value="0.17"/>
   <material name="red" >
@@ -24,5 +24,6 @@
         <origin xyz="0 0 0" rpy="0 0 0" />
         <geometry>
-          <box size="0.07 0.085 0.065" />
+          <!--box size="0.07 0.085 0.065" /-->
+          <mesh filename="package://ubiquitous_display_description/meshes/STL/ud_pt_base.stl" scale="0.001 0.001 0.001"/>
         </geometry>
         <material name="gray"/>
@@ -39,7 +40,8 @@
     <link name="${name}plate_link">
       <visual>
-        <origin xyz="0.075 0 0" rpy="0 0 0" />
+        <origin xyz="0 0 0" rpy="0 0 0" />
         <geometry>
-          <box size="0.35 0.095 0.003" />
+          <!--box size="0.35 0.095 0.003" /-->
+          <mesh filename="package://ubiquitous_display_description/meshes/STL/ud_pt_pan.stl" scale="0.001 0.001 0.001"/>
         </geometry>
         <material name="gray"/>
@@ -54,5 +56,5 @@
      </inertial>
     </link>
-    <link name="left_pt_pillars" >
+    <!--link name="left_pt_pillars" >
       <visual>
         <origin xyz="0 0 0" rpy="0 0 0" />
@@ -87,10 +89,11 @@
 	    izz="1.0"/>
      </inertial>
-    </link>
+   </link-->
     <link name="${name}projector_link">
       <visual>
-        <origin xyz="0.07 0.037 0" rpy="0 0 0" />
+        <origin xyz="0 0 0" rpy="0 0 0" />
         <geometry>
-          <box size="0.24 0.17 0.07" />
+          <!--box size="0.24 0.17 0.07" /-->
+          <mesh filename="package://ubiquitous_display_description/meshes/STL/ud_pt_tilt_with_projector.stl" scale="0.001 0.001 0.001"/>
         </geometry>
         <material name="gray"/>
@@ -126,5 +129,5 @@
       <dynamics damping="0.7"/>
     </joint>
-    <joint name="${name}plate_link_to_left_pt_pillars" type="fixed">
+    <!--joint name="${name}plate_link_to_left_pt_pillars" type="fixed">
       <parent link="${name}plate_link"/>
       <child link="left_pt_pillars"/>
@@ -135,5 +138,5 @@
       <child link="right_pt_pillars"/>
       <origin xyz="0.24 0 0.1" rpy="0 0 0" />
-    </joint>
+    </joint-->
     <joint name="tilt_joint" type="revolute">
       <parent link="${name}plate_link"/>

Commit message: [Fix] inertial tag in body

File: urdf/body/body.urdf.xacro (robot description, xacro)
@@ -19,4 +19,8 @@
   <xacro:property name="hokuyo_offset_x" value="-0.05"/>
   <xacro:property name="hokuyo_offset_z" value="0.037"/>
+  <!-- for inertial tag -->
+  <xacro:property name="bottom_pillars_mass" value="0.203"/>
+  <xacro:property name="middle_pillars_mass" value="0.509"/>
+  <xacro:property name="top_pillars_mass" value="0.672"/>
   <!-- Definition of colors -->
   <material name="black">
@@ -35,4 +39,12 @@
       <material name="black"/>
     </visual>
+    <!-- <inertial>
+      <origin xyz="0 0 0" rpy="0 0 0"/>
+      <mass value="0.5"/>
+      <inertia
+     ixx="2.666E+06" ixy="2.666E+06" ixz="2.124E+04"
+     iyx="2.666E+06" iyy="2.124E+04" iyz="2.666E+06"
+     izx="2.124E+04" izy="2.666E+06" izz="2.666E+06"/>
+    </inertial> -->
   </xacro:macro>
   <xacro:macro name="plate_template" params="name">
@@ -47,4 +59,12 @@
       </visual>
     </link>
+    <!-- <inertial>
+      <origin xyz="0 0 0" rpy="0 0 0"/>
+      <mass value="1.0"/>
+      <inertia
+     ixx="3.167E+06" ixy="2.269E+07" ixz="1.953E+07"
+     iyx="2.269E+07" iyy="1.953E+07" iyz="3.167E+06"
+     izx="1.953E+07" izy="3.167E+06" izz="2.269E+07"/>
+    </inertial> -->
   </xacro:macro>
   <xacro:macro name="tower_template" params="name pillar_height">

Commit message: [Fix] ppantilt and body inertial tag

File: urdf/body/body.urdf.xacro (robot description, xacro)
@@ -39,12 +39,12 @@
       <material name="black"/>
     </visual>
-    <!-- <inertial>
+    <inertial>
       <origin xyz="0 0 0" rpy="0 0 0"/>
       <mass value="0.5"/>
       <inertia
-     ixx="2.666E+06" ixy="2.666E+06" ixz="2.124E+04"
-     iyx="2.666E+06" iyy="2.124E+04" iyz="2.666E+06"
-     izx="2.124E+04" izy="2.666E+06" izz="2.666E+06"/>
-    </inertial> -->
+     ixx="0.0018" ixy="0" ixz="0"
+     iyx="0" iyy="0.0018" iyz="0"
+     izx="0" izy="0" izz="0.000025"/>
+    </inertial>
   </xacro:macro>
   <xacro:macro name="plate_template" params="name">
@@ -59,12 +59,12 @@
       </visual>
     </link>
-    <!-- <inertial>
+    <inertial>
       <origin xyz="0 0 0" rpy="0 0 0"/>
       <mass value="1.0"/>
       <inertia
-     ixx="3.167E+06" ixy="2.269E+07" ixz="1.953E+07"
-     iyx="2.269E+07" iyy="1.953E+07" iyz="3.167E+06"
-     izx="1.953E+07" izy="3.167E+06" izz="2.269E+07"/>
-    </inertial> -->
+     ixx="0.0211" ixy="0" ixz="0"
+     iyx="0" iyy="0.0036" iyz="0"
+     izx="0" izy="0" izz="0.0241"/>
+    </inertial>
   </xacro:macro>
   <xacro:macro name="tower_template" params="name pillar_height">

File: urdf/pantilt/pantilt.urdf.xacro (robot description, xacro)
@@ -29,5 +29,5 @@
      <inertial>
        <origin xyz="0 0 ${base_to_box_height/2}" rpy="0 0 0"/>
-       <mass value="0.28"/>
+       <mass value="0.78"/>
        <inertia
 	    ixx="0.00190" ixy="0.0" ixz="0.0"
@@ -47,5 +47,5 @@
      <inertial>
        <origin xyz="0 0 0.0015" rpy="0 0 0"/>
-       <mass value="0.08"/>
+       <mass value="1.5"/>
        <inertia
 	    ixx="0.00150" ixy="0.0" ixz="0.0"
@@ -65,5 +65,5 @@
      <inertial>
        <origin xyz="0 0 0" rpy="0 0 0"/>
-       <mass value="2"/>
+       <mass value="1.3"/>
        <inertia
 	    ixx="0.00536" ixy="0.0" ixz="0.0"
