Commit message: [Add] utm-30lx.gazebo.xacro

File: urdf/sensor/lrf/hokuyo_utm30lx.gazebo.xacro (robot description, xacro)
@@ -1,36 +1,73 @@
 <?xml version="1.0"?>
 <robot xmlns:xacro="http://ros.org/wiki/xacro">
-  <xacro:macro name="hokuyo_utm30lx_gazebo" params="prefix min_rad max_rad min_range max_range">
-	<gazebo reference="${prefix}_laser_frame">
-      <sensor type="ray" name="${prefix}_lrf_sensor">
-		<pose>0 0 0 0 0 0</pose>
-		<visualize>true</visualize>
-		<update_rate>40</update_rate>
-		<ray>
+  <xacro:macro name="hokuyo_utm30lx_gazebo" params="name ray_count min_angle max_angle">
+    <gazebo reference="${name}_laser_frame">
+      <sensor type="ray" name="${name}">
+        <always_on>true</always_on>
+        <update_rate>40</update_rate>
+        <pose>0 0 0 0 0 0</pose>
+        <visualize>false</visualize>
+        <ray>
           <scan>
-			<horizontal>
-              <samples>720</samples>
+            <horizontal>
+              <samples>${ray_count}</samples>
               <resolution>1</resolution>
-              <min_angle>${min_rad}</min_angle>
-              <max_angle>${max_rad}</max_angle>
-			</horizontal>
+              <min_angle>${min_angle * M_PI/180}</min_angle>
+              <max_angle>${max_angle * M_PI/180}</max_angle>
+            </horizontal>
           </scan>
           <range>
-			<min>${min_range}</min>
-			<max>${max_range}</max>
-			<resolution>0.01</resolution>
+            <min>0.2</min>
+            <resolution>0.01</resolution>
+            <max>30.0</max>
           </range>
           <noise>
-			<type>gaussian</type>
-			<mean>0.0</mean>
-			<stddev>0.03</stddev>
+            <type>gaussian</type>
+            <mean>0.0</mean>
+            <stddev>0.004</stddev>
           </noise>
-		</ray>
-		<plugin name="gazebo_ros_${prefix}_lrf_controller" filename="libgazebo_ros_laser.so">
-          <topicName>${prefix}_scan</topicName>
-          <frameName>${prefix}_laser_frame</frameName>
-		</plugin>
+        </ray>
+        <plugin name="gazebo_ros_${name}_controller" filename="libgazebo_ros_laser.so">
+          <topicName>${name}_scan</topicName>
+          <frameName>${name}_laser_frame</frameName>
+        </plugin>
       </sensor>
-	</gazebo>
+    </gazebo>
+  </xacro:macro>
+  <xacro:macro name="hokuyo_utm30lx_gpu" params="name parent *origin ros_topic update_rate ray_count min_angle max_angle">
+    <xacro:hokuyo_utm30lx_model name="${name}" parent="${parent}">
+      <!--xacro:insert_block name="origin" /-->
+    </xacro:hokuyo_utm30lx_model>
+    <gazebo reference="${name}_frame">
+      <sensor type="gpu_ray" name="${name}">
+        <update_rate>${update_rate}</update_rate>
+        <pose>0 0 0 0 0 0</pose>
+        <visualize>false</visualize>
+        <ray>
+          <scan>
+            <horizontal>
+              <samples>${ray_count}</samples>
+              <resolution>1</resolution>
+              <min_angle>${min_angle * M_PI/180}</min_angle>
+              <max_angle>${max_angle * M_PI/180}</max_angle>
+            </horizontal>
+          </scan>
+          <range>
+            <min>0.2</min>
+            <max>30.0</max>
+            <resolution>0.01</resolution>
+          </range>
+          <noise>
+            <type>gaussian</type>
+            <mean>0.0</mean>
+            <stddev>0.004</stddev>
+          </noise>
+        </ray>
+        <plugin name="gazebo_ros_${name}_controller" filename="libgazebo_ros_gpu_laser.so">
+          <topicName>${ros_topic}</topicName>
+          <frameName>${name}_frame</frameName>
+        </plugin>
+      </sensor>
+    </gazebo>
   </xacro:macro>
 </robot>

File: urdf/sensor/lrf/hokuyo_utm30lx.urdf.xacro (robot description, xacro)
@@ -30,77 +30,5 @@
         </collision>
       </link>
-    </xacro:macro>
-    <xacro:macro name="hokuyo_utm30lx" params="name parent *origin ros_topic update_rate ray_count min_angle max_angle">
-      <xacro:hokuyo_utm30lx_model name="${name}" parent="${parent}">
-        <!--xacro:insert_block name="origin" /-->
-      </xacro:hokuyo_utm30lx_model>
-      <gazebo reference="${name}_frame">
-        <sensor type="ray" name="${name}">
-          <always_on>true</always_on>
-          <update_rate>${update_rate}</update_rate>
-          <pose>0 0 0 0 0 0</pose>
-          <visualize>false</visualize>
-          <ray>
-            <scan>
-              <horizontal>
-                <samples>${ray_count}</samples>
-                <resolution>1</resolution>
-                <min_angle>${min_angle * M_PI/180}</min_angle>
-                <max_angle>${max_angle * M_PI/180}</max_angle>
-              </horizontal>
-            </scan>
-            <range>
-              <min>0.2</min>
-              <max>30.0</max>
-              <resolution>0.01</resolution>
-            </range>
-            <noise>
-              <type>gaussian</type>
-              <mean>0.0</mean>
-              <stddev>0.004</stddev>
-            </noise>
-          </ray>
-          <plugin name="gazebo_ros_${name}_controller" filename="libgazebo_ros_laser.so">
-            <topicName>${ros_topic}</topicName>
-            <frameName>${name}_frame</frameName>
-          </plugin>
-        </sensor>
-      </gazebo>
-    </xacro:macro>
-    <xacro:macro name="hokuyo_utm30lx_gpu" params="name parent *origin ros_topic update_rate ray_count min_angle max_angle">
-      <xacro:hokuyo_utm30lx_model name="${name}" parent="${parent}">
-        <!--xacro:insert_block name="origin" /-->
-      </xacro:hokuyo_utm30lx_model>
-      <gazebo reference="${name}_frame">
-        <sensor type="gpu_ray" name="${name}">
-          <update_rate>${update_rate}</update_rate>
-          <pose>0 0 0 0 0 0</pose>
-          <visualize>false</visualize>
-          <ray>
-            <scan>
-              <horizontal>
-                <samples>${ray_count}</samples>
-                <resolution>1</resolution>
-                <min_angle>${min_angle * M_PI/180}</min_angle>
-                <max_angle>${max_angle * M_PI/180}</max_angle>
-              </horizontal>
-            </scan>
-            <range>
-              <min>0.2</min>
-              <max>30.0</max>
-              <resolution>0.01</resolution>
-            </range>
-            <noise>
-              <type>gaussian</type>
-              <mean>0.0</mean>
-              <stddev>0.004</stddev>
-            </noise>
-          </ray>
-          <plugin name="gazebo_ros_${name}_controller" filename="libgazebo_ros_gpu_laser.so">
-            <topicName>${ros_topic}</topicName>
-            <frameName>${name}_frame</frameName>
-          </plugin>
-        </sensor>
-      </gazebo>
+      <xacro:hokuyo_utm30lx_gazebo name="${name}" ray_count="1080" min_angle="0" max_angle="270" />
     </xacro:macro>
 </robot>

Commit message: [Fix] active gpu_ray

File: urdf/sensor/lrf/hokuyo_utm30lx.gazebo.xacro (robot description, xacro)
@@ -35,11 +35,8 @@
     </gazebo>
   </xacro:macro>
-  <xacro:macro name="hokuyo_utm30lx_gpu" params="name parent *origin ros_topic update_rate ray_count min_angle max_angle">
-    <xacro:hokuyo_utm30lx_model name="${name}" parent="${parent}">
-      <!--xacro:insert_block name="origin" /-->
-    </xacro:hokuyo_utm30lx_model>
+  <xacro:macro name="hokuyo_utm30lx_gpu" params="name ray_count min_angle max_angle">
     <gazebo reference="${name}_frame">
       <sensor type="gpu_ray" name="${name}">
-        <update_rate>${update_rate}</update_rate>
+        <update_rate>40</update_rate>
         <pose>0 0 0 0 0 0</pose>
         <visualize>false</visualize>
@@ -65,5 +62,5 @@
         </ray>
         <plugin name="gazebo_ros_${name}_controller" filename="libgazebo_ros_gpu_laser.so">
-          <topicName>${ros_topic}</topicName>
+          <topicName>${name}_scan</topicName>
           <frameName>${name}_frame</frameName>
         </plugin>

File: urdf/sensor/lrf/hokuyo_utm30lx.urdf.xacro (robot description, xacro)
@@ -30,5 +30,5 @@
         </collision>
       </link>
-      <xacro:hokuyo_utm30lx_gazebo name="${name}" ray_count="1080" min_angle="-135" max_angle="135" />
+      <xacro:hokuyo_utm30lx_gpu name="${name}" ray_count="1080" min_angle="-135" max_angle="135" />
     </xacro:macro>
 </robot>
